File: hardware/pcb/nrf8001.sch (KiCad schematic (older format))
At the start: 20 parts

Commit message: version 1 of layout
Parts:
- C1, C10, C11, C12, C13, C2, C3, C4, C5, C6, C7, C8, C9: renamed from C?; footprint (none) -> Capacitors_SMD:C_0402
- L1, L2, L3: renamed from L?; footprint (none) -> Capacitors_SMD:C_0402
- R1: renamed from R?; footprint (none) -> Resistors_SMD:R_0402
- U1: renamed from U?; footprint (none) -> Housings_DFN_QFN:QFN-32-1EP_5x5mm_Pitch0.5mm
- Y1: renamed from Y?; footprint (none) -> aero:FC-135R
- Y2: renamed from Y?; footprint (none) -> aero:crystal_SMD_3225
Connections:
- net RXD: now reaches U1.10 (RXD)
- net at U1.27 (XC2): now also C8.2, Y2.2
- net at C7.2, U1.28 (XC1), Y2.1: no longer C8.2, Y2.2

Commit message: pcb updates
Changed lines of the file:
@@
 $Descr A4 11693 8268
 encoding utf-8
-Sheet 2 2
+Sheet 2 3
 Title ""
 Date ""
@@
 	6950 3750 6950 2900
 Connection ~ 6950 2900
-Text HLabel 2050 1200 0    60   Input ~ 0
-Vcc
-Text HLabel 2050 1350 0    60   Input ~ 0
-Gnd
-$Comp
-L VCC #PWR018
-U 1 1 551C2314
-P 2350 1100
-F 0 "#PWR018" H 2350 950 50  0001 C CNN
-F 1 "VCC" H 2350 1250 50  0000 C CNN
-F 2 "" H 2350 1100 60  0000 C CNN
-F 3 "" H 2350 1100 60  0000 C CNN
-	1    2350 1100
-	1    0    0    -1
-$EndComp
-$Comp
-L GND #PWR019
-U 1 1 551C2350
-P 2350 1400
-F 0 "#PWR019" H 2350 1150 50  0001 C CNN
-F 1 "GND" H 2350 1250 50  0000 C CNN
-F 2 "" H 2350 1400 60  0000 C CNN
-F 3 "" H 2350 1400 60  0000 C CNN
-	1    2350 1400
-	1    0    0    -1
-$EndComp
-Wire Wire Line
-	2050 1350 2350 1350
-Wire Wire Line
-	2350 1350 2350 1400
-Wire Wire Line
-	2350 1100 2350 1200
-Wire Wire Line
-	2350 1200 2050 1200
 Text HLabel 5400 5350 3    60   Input ~ 0
 RXD

Commit message: Removed nRF8001 connections; beginning eventual design
Connections:
- net VCC renamed +3V3
Changed lines of the file:
@@
-$EndComp
-$Comp
-L VCC #PWR04
-U 1 1 551C0D8A
-P 2650 3550
-F 0 "#PWR04" H 2650 3400 50  0001 C CNN
-F 1 "VCC" H 2650 3700 50  0000 C CNN
-F 2 "" H 2650 3550 60  0000 C CNN
-F 3 "" H 2650 3550 60  0000 C CNN
-	1    2650 3550
-	1    0    0    -1
 $EndComp
 $Comp
@@
 $EndComp
 $Comp
-L GND #PWR05
+L GND #PWR04
 U 1 1 551C1217
 P 2350 5800
-F 0 "#PWR05" H 2350 5550 50  0001 C CNN
+F 0 "#PWR04" H 2350 5550 50  0001 C CNN
 F 1 "GND" H 2350 5650 50  0000 C CNN
 F 2 "" H 2350 5800 60  0000 C CNN
@@
 $EndComp
 $Comp
-L GND #PWR06
+L GND #PWR05
 U 1 1 551C134D
 P 4700 4500
-F 0 "#PWR06" H 4700 4250 50  0001 C CNN
+F 0 "#PWR05" H 4700 4250 50  0001 C CNN
 F 1 "GND" H 4700 4350 50  0000 C CNN
 F 2 "" H 4700 4500 60  0000 C CNN
@@
 $EndComp
 $Comp
-L VCC #PWR07
-U 1 1 551C13BA
-P 5050 4950
-F 0 "#PWR07" H 5050 4800 50  0001 C CNN
-F 1 "VCC" H 5050 5100 50  0000 C CNN
-F 2 "" H 5050 4950 60  0000 C CNN
-F 3 "" H 5050 4950 60  0000 C CNN
-	1    5050 4950
-	1    0    0    -1
-$EndComp
-$Comp
-L GND #PWR08
+L GND #PWR06
 U 1 1 551C13DC
 P 5050 5400
-F 0 "#PWR08" H 5050 5150 50  0001 C CNN
+F 0 "#PWR06" H 5050 5150 50  0001 C CNN
 F 1 "GND" H 5050 5250 50  0000 C CNN
 F 2 "" H 5050 5400 60  0000 C CNN
@@
 $EndComp
 $Comp
-L GND #PWR09
+L GND #PWR07
 U 1 1 551C159D
 P 5150 2950
-F 0 "#PWR09" H 5150 2700 50  0001 C CNN
+F 0 "#PWR07" H 5150 2700 50  0001 C CNN
 F 1 "GND" H 5150 2800 50  0000 C CNN
 F 2 "" H 5150 2950 60  0000 C CNN
 F 3 "" H 5150 2950 60  0000 C CNN
 	1    5150 2950
-	1    0    0    -1
-$EndComp
-$Comp
-L VCC #PWR010
-U 1 1 551C167B
-P 5600 2900
-F 0 "#PWR010" H 5600 2750 50  0001 C CNN
-F 1 "VCC" H 5600 3050 50  0000 C CNN
-F 2 "" H 5600 2900 60  0000 C CNN
-F 3 "" H 5600 2900 60  0000 C CNN
-	1    5600 2900
 	1    0    0    -1
 $EndComp
@@
 $EndComp
 $Comp
-L GND #PWR011
+L GND #PWR08
 U 1 1 551C18D0
 P 7550 2150
-F 0 "#PWR011" H 7550 1900 50  0001 C CNN
+F 0 "#PWR08" H 7550 1900 50  0001 C CNN
 F 1 "GND" H 7550 2000 50  0000 C CNN
 F 2 "" H 7550 2150 60  0000 C CNN
@@
 $EndComp
 $Comp
-L GND #PWR012
+L GND #PWR09
 U 1 1 551C1EC5
 P 7200 3000
-F 0 "#PWR012" H 7200 2750 50  0001 C CNN
+F 0 "#PWR09" H 7200 2750 50  0001 C CNN
 F 1 "GND" H 7200 2850 50  0000 C CNN
 F 2 "" H 7200 3000 60  0000 C CNN
 F 3 "" H 7200 3000 60  0000 C CNN
 	1    7200 3000
-	1    0    0    -1
-$EndComp
-$Comp
-L VCC #PWR013
-U 1 1 551C1FEA
-P 7200 2550
-F 0 "#PWR013" H 7200 2400 50  0001 C CNN
-F 1 "VCC" H 7200 2700 50  0000 C CNN
-F 2 "" H 7200 2550 60  0000 C CNN
-F 3 "" H 7200 2550 60  0000 C CNN
-	1    7200 2550
 	1    0    0    -1
 $EndComp
@@
 NoConn ~ 5900 4800
 $Comp
-L GND #PWR014
+L GND #PWR010
 U 1 1 551C247D
 P 6550 4450
-F 0 "#PWR014" H 6550 4200 50  0001 C CNN
+F 0 "#PWR010" H 6550 4200 50  0001 C CNN
 F 1 "GND" H 6550 4300 50  0000 C CNN
 F 2 "" H 6550 4450 60  0000 C CNN
@@
 $EndComp
 $Comp
-L GND #PWR015
+L GND #PWR011
 U 1 1 551C26C3
 P 8200 5100
-F 0 "#PWR015" H 8200 4850 50  0001 C CNN
+F 0 "#PWR011" H 8200 4850 50  0001 C CNN
 F 1 "GND" H 8200 4950 50  0000 C CNN
 F 2 "" H 8200 5100 60  0000 C CNN
@@
 $EndComp
 $Comp
-L GND #PWR016
+L GND #PWR012
 U 1 1 551C26F1
 P 8500 5100
-F 0 "#PWR016" H 8500 4850 50  0001 C CNN
+F 0 "#PWR012" H 8500 4850 50  0001 C CNN
 F 1 "GND" H 8500 4950 50  0000 C CNN
 F 2 "" H 8500 5100 60  0000 C CNN
@@
 $EndComp
 $Comp
-L GND #PWR017
+L GND #PWR013
 U 1 1 551C3732
 P 9700 4400
-F 0 "#PWR017" H 9700 4150 50  0001 C CNN
+F 0 "#PWR013" H 9700 4150 50  0001 C CNN
 F 1 "GND" H 9700 4250 50  0000 C CNN
 F 2 "" H 9700 4400 60  0000 C CNN
@@
 Wire Wire Line
 	5800 1950 6850 1950
+$Comp
+L +3V #PWR014
+U 1 1 55282769
+P 2650 3550
+F 0 "#PWR014" H 2650 3450 60  0001 C CNN
+F 1 "+3V" H 2500 3700 60  0000 C CNN
+F 2 "" H 2650 3550 60  0000 C CNN
+F 3 "" H 2650 3550 60  0000 C CNN
+	1    2650 3550
+	1    0    0    -1
+$EndComp
+$Comp
+L +3V #PWR015
+U 1 1 5528286C
+P 5050 4950
+F 0 "#PWR015" H 5050 4850 60  0001 C CNN
+F 1 "+3V" H 4900 5100 60  0000 C CNN
+F 2 "" H 5050 4950 60  0000 C CNN
+F 3 "" H 5050 4950 60  0000 C CNN
+	1    5050 4950
+	1    0    0    -1
+$EndComp
+$Comp
+L +3V #PWR016
+U 1 1 552829BF
+P 5600 2900
+F 0 "#PWR016" H 5600 2800 60  0001 C CNN
+F 1 "+3V" H 5450 3050 60  0000 C CNN
+F 2 "" H 5600 2900 60  0000 C CNN
+F 3 "" H 5600 2900 60  0000 C CNN
+	1    5600 2900
+	1    0    0    -1
+$EndComp
+$Comp
+L +3V #PWR017
+U 1 1 55282B5E
+P 7200 2550
+F 0 "#PWR017" H 7200 2450 60  0001 C CNN
+F 1 "+3V" H 7050 2700 60  0000 C CNN
+F 2 "" H 7200 2550 60  0000 C CNN
+F 3 "" H 7200 2550 60  0000 C CNN
+	1    7200 2550
+	1    0    0    -1
+$EndComp
 $EndSCHEMATC
