File: hardware/pcb/nrf8001.sch (KiCad schematic (older format))
At the start: 20 parts, among them U1 nRF8001, Y1 32.768KHz, Y2 16MHz

Commit message: more changes
Parts:
- L2: footprint Capacitors_SMD:C_0402 -> (none)
- renumbered C1 to C11, C2 to C12, C3 to C13, C4 to C14, C5 to C15, C6 to C16, C7 to C17, C8 to C18, C9 to C19, C10 to C20, C11 to C21, C12 to C22, C13 to C23, R1 to R5, U1 to U2, Y1 to Y3, Y2 to Y4
Changed lines of the file:
@@
 $EndDescr
 $Comp
-L nRF8001 U1
+L nRF8001 U2
 U 1 1 551C0A1A
 P 5550 4050
-F 0 "U1" H 6200 3450 60  0000 C CNN
+F 0 "U2" H 6200 3450 60  0000 C CNN
 F 1 "nRF8001" H 5650 4150 60  0000 C CNN
 F 2 "Housings_DFN_QFN:QFN-32-1EP_5x5mm_Pitch0.5mm" H 7650 3600 60  0001 C CNN
@@
 $EndComp
 $Comp
-L C C1
+L C C11
 U 1 1 551C0AC5
 P 2650 4200
-F 0 "C1" H 2675 4300 50  0000 L CNN
+F 0 "C11" H 2675 4300 50  0000 L CNN
 F 1 "100nF" H 2675 4100 50  0000 L CNN
 F 2 "Capacitors_SMD:C_0402" H 2688 4050 30  0001 C CNN
@@
 $EndComp
 $Comp
-L C C2
+L C C12
 U 1 1 551C0AEF
 P 2950 4200
-F 0 "C2" H 2975 4300 50  0000 L CNN
+F 0 "C12" H 2975 4300 50  0000 L CNN
 F 1 "100nF" H 2975 4100 50  0000 L CNN
 F 2 "Capacitors_SMD:C_0402" H 2988 4050 30  0001 C CNN
@@
 $EndComp
 $Comp
-L C C5
+L C C15
 U 1 1 551C0B13
 P 3250 4200
-F 0 "C5" H 3275 4300 50  0000 L CNN
+F 0 "C15" H 3275 4300 50  0000 L CNN
 F 1 "33nF" H 3275 4100 50  0000 L CNN
 F 2 "Capacitors_SMD:C_0402" H 3288 4050 30  0001 C CNN
@@
 $EndComp
 $Comp
-L GND #PWR09
+L GND #PWR18
 U 1 1 551C0C1E
 P 2650 4400
-F 0 "#PWR09" H 2650 4150 50  0001 C CNN
+F 0 "#PWR18" H 2650 4150 50  0001 C CNN
 F 1 "GND" H 2650 4250 50  0000 C CNN
 F 2 "" H 2650 4400 60  0000 C CNN
@@
 $EndComp
 $Comp
-L GND #PWR010
+L GND #PWR19
 U 1 1 551C0C3A
 P 2950 4400
-F 0 "#PWR010" H 2950 4150 50  0001 C CNN
+F 0 "#PWR19" H 2950 4150 50  0001 C CNN
 F 1 "GND" H 2950 4250 50  0000 C CNN
 F 2 "" H 2950 4400 60  0000 C CNN
@@
 $EndComp
 $Comp
-L GND #PWR011
+L GND #PWR20
 U 1 1 551C0D06
 P 3250 4400
-F 0 "#PWR011" H 3250 4150 50  0001 C CNN
+F 0 "#PWR20" H 3250 4150 50  0001 C CNN
 F 1 "GND" H 3250 4250 50  0000 C CNN
 F 2 "" H 3250 4400 60  0000 C CNN
@@
 $EndComp
 $Comp
-L Crystal Y1
+L Crystal Y3
 U 1 1 551C0F7F
 P 3600 5350
-F 0 "Y1" H 3600 5500 50  0000 C CNN
+F 0 "Y3" H 3600 5500 50  0000 C CNN
 F 1 "32.768KHz" H 3600 5200 50  0000 C CNN
 F 2 "aero:FC-135R" H 3600 5350 60  0001 C CNN
@@
 $EndComp
 $Comp
-L C C3
+L C C13
 U 1 1 551C1027
 P 3000 5050
-F 0 "C3" H 3025 5150 50  0000 L CNN
+F 0 "C13" H 3025 5150 50  0000 L CNN
 F 1 "15pF" H 3025 4950 50  0000 L CNN
 F 2 "Capacitors_SMD:C_0402" H 3038 4900 30  0001 C CNN
@@
 $EndComp
 $Comp
-L C C4
+L C C14
 U 1 1 551C108E
 P 3000 5700
-F 0 "C4" H 3025 5800 50  0000 L CNN
+F 0 "C14" H 3025 5800 50  0000 L CNN
 F 1 "15pF" H 3025 5600 50  0000 L CNN
 F 2 "Capacitors_SMD:C_0402" H 3038 5550 30  0001 C CNN
@@
 $EndComp
 $Comp
-L GND #PWR012
+L GND #PWR16
 U 1 1 551C1217
 P 2350 5800
-F 0 "#PWR012" H 2350 5550 50  0001 C CNN
+F 0 "#PWR16" H 2350 5550 50  0001 C CNN
 F 1 "GND" H 2350 5650 50  0000 C CNN
 F 2 "" H 2350 5800 60  0000 C CNN
@@
 $EndComp
 $Comp
-L GND #PWR013
+L GND #PWR21
 U 1 1 551C134D
 P 4700 4500
-F 0 "#PWR013" H 4700 4250 50  0001 C CNN
+F 0 "#PWR21" H 4700 4250 50  0001 C CNN
 F 1 "GND" H 4700 4350 50  0000 C CNN
 F 2 "" H 4700 4500 60  0000 C CNN
@@
 $EndComp
 $Comp
-L GND #PWR014
+L GND #PWR23
 U 1 1 551C13DC
 P 5050 5400
-F 0 "#PWR014" H 5050 5150 50  0001 C CNN
+F 0 "#PWR23" H 5050 5150 50  0001 C CNN
 F 1 "GND" H 5050 5250 50  0000 C CNN
 F 2 "" H 5050 5400 60  0000 C CNN
@@
 $EndComp
 $Comp
-L C C6
+L C C16
 U 1 1 551C140C
 P 5050 5250
-F 0 "C6" H 5075 5350 50  0000 L CNN
+F 0 "C16" H 5075 5350 50  0000 L CNN
 F 1 "100nF" H 5075 5150 50  0000 L CNN
 F 2 "Capacitors_SMD:C_0402" H 5088 5100 30  0001 C CNN
@@
 $EndComp
 $Comp
-L GND #PWR015
+L GND #PWR24
 U 1 1 551C159D
 P 5150 2950
-F 0 "#PWR015" H 5150 2700 50  0001 C CNN
+F 0 "#PWR24" H 5150 2700 50  0001 C CNN
 F 1 "GND" H 5150 2800 50  0000 C CNN
 F 2 "" H 5150 2950 60  0000 C CNN
@@
 $EndComp
 $Comp
-L Crystal Y2
+L Crystal Y4
 U 1 1 551C1703
 P 6450 1600
-F 0 "Y2" H 6450 1750 50  0000 C CNN
+F 0 "Y4" H 6450 1750 50  0000 C CNN
 F 1 "16MHz" H 6450 1450 50  0000 C CNN
 F 2 "aero:crystal_SMD_3225" H 6450 1600 60  0001 C CNN
@@
 $EndComp
 $Comp
-L C C7
+L C C17
 U 1 1 551C17DD
 P 7000 1250
-F 0 "C7" H 7025 1350 50  0000 L CNN
+F 0 "C17" H 7025 1350 50  0000 L CNN
 F 1 "12pF" H 7025 1150 50  0000 L CNN
 F 2 "Capacitors_SMD:C_0402" H 7038 1100 30  0001 C CNN
@@
 $EndComp
 $Comp
-L C C8
+L C C18
 U 1 1 551C1811
 P 7000 1950
-F 0 "C8" H 7025 2050 50  0000 L CNN
+F 0 "C18" H 7025 2050 50  0000 L CNN
 F 1 "12pF" H 7025 1850 50  0000 L CNN
 F 2 "Capacitors_SMD:C_0402" H 7038 1800 30  0001 C CNN
@@
 $EndComp
 $Comp
-L GND #PWR016
+L GND #PWR29
 U 1 1 551C18D0
 P 7550 2150
-F 0 "#PWR016" H 7550 1900 50  0001 C CNN
+F 0 "#PWR29" H 7550 1900 50  0001 C CNN
 F 1 "GND" H 7550 2000 50  0000 C CNN
 F 2 "" H 7550 2150 60  0000 C CNN
@@
 $EndComp
 $Comp
-L R R1
+L R R5
 U 1 1 551C1DE2
 P 6450 2900
-F 0 "R1" V 6530 2900 50  0000 C CNN
+F 0 "R5" V 6530 2900 50  0000 C CNN
 F 1 "22k" V 6450 2900 50  0000 C CNN
 F 2 "Resistors_SMD:R_0402" V 6380 2900 30  0001 C CNN
@@
 $EndComp
 $Comp
-L GND #PWR017
+L GND #PWR28
 U 1 1 551C1EC5
 P 7200 3000
-F 0 "#PWR017" H 7200 2750 50  0001 C CNN
+F 0 "#PWR28" H 7200 2750 50  0001 C CNN
 F 1 "GND" H 7200 2850 50  0000 C CNN
 F 2 "" H 7200 3000 60  0000 C CNN
@@
 $EndComp
 $Comp
-L C C9
+L C C19
 U 1 1 551C2016
 P 7200 2750
-F 0 "C9" H 7225 2850 50  0000 L CNN
+F 0 "C19" H 7225 2850 50  0000 L CNN
 F 1 "1.0nF" H 7225 2650 50  0000 L CNN
 F 2 "Capacitors_SMD:C_0402" H 7238 2600 30  0001 C CNN
@@
 NoConn ~ 5900 4800
 $Comp
-L GND #PWR018
+L GND #PWR26
 U 1 1 551C247D
 P 6550 4450
-F 0 "#PWR018" H 6550 4200 50  0001 C CNN
+F 0 "#PWR26" H 6550 4200 50  0001 C CNN
 F 1 "GND" H 6550 4300 50  0000 C CNN
 F 2 "" H 6550 4450 60  0000 C CNN
@@
 $EndComp
 $Comp
-L GND #PWR019
+L GND #PWR30
 U 1 1 551C26C3
 P 8200 5100
-F 0 "#PWR019" H 8200 4850 50  0001 C CNN
+F 0 "#PWR30" H 8200 4850 50  0001 C CNN
 F 1 "GND" H 8200 4950 50  0000 C CNN
 F 2 "" H 8200 5100 60  0000 C CNN
@@
 $EndComp
 $Comp
-L GND #PWR020
+L GND #PWR31
 U 1 1 551C26F1
 P 8500 5100
-F 0 "#PWR020" H 8500 4850 50  0001 C CNN
+F 0 "#PWR31" H 8500 4850 50  0001 C CNN
 F 1 "GND" H 8500 4950 50  0000 C CNN
 F 2 "" H 8500 5100 60  0000 C CNN
@@
 $EndComp
 $Comp
-L C C10
+L C C20
 U 1 1 551C277F
 P 8200 4950
-F 0 "C10" H 8225 5050 50  0000 L CNN
+F 0 "C20" H 8225 5050 50  0000 L CNN
 F 1 "2.2nF" H 8225 4850 50  0000 L CNN
 F 2 "Capacitors_SMD:C_0402" H 8238 4800 30  0001 C CNN
@@
 $EndComp
 $Comp
-L C C11
+L C C21
 U 1 1 551C27BB
 P 8500 4950
-F 0 "C11" H 8525 5050 50  0000 L CNN
+F 0 "C21" H 8525 5050 50  0000 L CNN
 F 1 "NC" H 8525 4850 50  0000 L CNN
 F 2 "Capacitors_SMD:C_0402" H 8538 4800 30  0001 C CNN
@@
 F 0 "L2" V 8050 3750 50  0000 C CNN
 F 1 "3.9nH" V 8200 3750 50  0000 C CNN
-F 2 "Capacitors_SMD:C_0402" H 8100 3750 60  0001 C CNN
+F 2 "" H 8100 3750 60  0001 C CNN
 F 3 "" H 8100 3750 60  0000 C CNN
 	1    8100 3750
@@
 $EndComp
 $Comp
-L C C12
+L C C22
 U 1 1 551C2C8B
 P 9000 3750
-F 0 "C12" H 9025 3850 50  0000 L CNN
+F 0 "C22" H 9025 3850 50  0000 L CNN
 F 1 "1.8pF" H 9025 3650 50  0000 L CNN
 F 2 "Capacitors_SMD:C_0402" H 9038 3600 30  0001 C CNN
@@
 $EndComp
 $Comp
-L C C13
+L C C23
 U 1 1 551C3165
 P 9700 4100
-F 0 "C13" H 9725 4200 50  0000 L CNN
+F 0 "C23" H 9725 4200 50  0000 L CNN
 F 1 "1.2pF" H 9725 4000 50  0000 L CNN
 F 2 "Capacitors_SMD:C_0402" H 9738 3950 30  0001 C CNN
@@
 $EndComp
 $Comp
-L GND #PWR021
+L GND #PWR32
 U 1 1 551C3732
 P 9700 4400
-F 0 "#PWR021" H 9700 4150 50  0001 C CNN
+F 0 "#PWR32" H 9700 4150 50  0001 C CNN
 F 1 "GND" H 9700 4250 50  0000 C CNN
 F 2 "" H 9700 4400 60  0000 C CNN
@@
 RXD
 Wire Wire Line
-	5400 5350 5400 4800
-Wire Wire Line
 	5800 3150 5800 1950
 Wire Wire Line
 	5800 1950 6850 1950
 $Comp
-L +3V #PWR022
+L +3V #PWR17
 U 1 1 55282769
 P 2650 3550
-F 0 "#PWR022" H 2650 3450 60  0001 C CNN
+F 0 "#PWR17" H 2650 3450 60  0001 C CNN
 F 1 "+3V" H 2500 3700 60  0000 C CNN
 F 2 "" H 2650 3550 60  0000 C CNN
@@
 $EndComp
 $Comp
-L +3V #PWR023
+L +3V #PWR22
 U 1 1 5528286C
 P 5050 4950
-F 0 "#PWR023" H 5050 4850 60  0001 C CNN
+F 0 "#PWR22" H 5050 4850 60  0001 C CNN
 F 1 "+3V" H 4900 5100 60  0000 C CNN
 F 2 "" H 5050 4950 60  0000 C CNN
@@
 $EndComp
 $Comp
-L +3V #PWR024
+L +3V #PWR25
 U 1 1 552829BF
 P 5600 2900
-F 0 "#PWR024" H 5600 2800 60  0001 C CNN
+F 0 "#PWR25" H 5600 2800 60  0001 C CNN
 F 1 "+3V" H 5450 3050 60  0000 C CNN
 F 2 "" H 5600 2900 60  0000 C CNN
@@
 $EndComp
 $Comp
-L +3V #PWR025
+L +3V #PWR27
 U 1 1 55282B5E
 P 7200 2550
-F 0 "#PWR025" H 7200 2450 60  0001 C CNN
+F 0 "#PWR27" H 7200 2450 60  0001 C CNN
 F 1 "+3V" H 7050 2700 60  0000 C CNN
 F 2 "" H 7200 2550 60  0000 C CNN
@@
 	1    0    0    -1
 $EndComp
+Wire Wire Line
+	5400 4800 5400 5350
 $EndSCHEMATC

Commit message: mega commit
Parts:
- C11, C12, C13, C14, C15, C16, C17, C18, C19, C20, C21, C22, C23, L1, L3: footprint Capacitors_SMD:C_0402 -> Capacitors_SMD:C_0603
- L2: footprint (none) -> Capacitors_SMD:C_0603
- R6: renamed from R5; footprint Resistors_SMD:R_0402 -> Resistors_SMD:R_0603
Changed lines of the file:
@@
 F 0 "C11" H 2675 4300 50  0000 L CNN
 F 1 "100nF" H 2675 4100 50  0000 L CNN
-F 2 "Capacitors_SMD:C_0402" H 2688 4050 30  0001 C CNN
+F 2 "Capacitors_SMD:C_0603" H 2688 4050 30  0001 C CNN
 F 3 "" H 2650 4200 60  0000 C CNN
 	1    2650 4200
@@
 F 0 "C12" H 2975 4300 50  0000 L CNN
 F 1 "100nF" H 2975 4100 50  0000 L CNN
-F 2 "Capacitors_SMD:C_0402" H 2988 4050 30  0001 C CNN
+F 2 "Capacitors_SMD:C_0603" H 2988 4050 30  0001 C CNN
 F 3 "" H 2950 4200 60  0000 C CNN
 	1    2950 4200
@@
 F 0 "C15" H 3275 4300 50  0000 L CNN
 F 1 "33nF" H 3275 4100 50  0000 L CNN
-F 2 "Capacitors_SMD:C_0402" H 3288 4050 30  0001 C CNN
+F 2 "Capacitors_SMD:C_0603" H 3288 4050 30  0001 C CNN
 F 3 "" H 3250 4200 60  0000 C CNN
 	1    3250 4200
@@
 $EndComp
 $Comp
-L GND #PWR18
+L GND #PWR017
 U 1 1 551C0C1E
 P 2650 4400
-F 0 "#PWR18" H 2650 4150 50  0001 C CNN
+F 0 "#PWR017" H 2650 4150 50  0001 C CNN
 F 1 "GND" H 2650 4250 50  0000 C CNN
 F 2 "" H 2650 4400 60  0000 C CNN
@@
 $EndComp
 $Comp
-L GND #PWR19
+L GND #PWR018
 U 1 1 551C0C3A
 P 2950 4400
-F 0 "#PWR19" H 2950 4150 50  0001 C CNN
+F 0 "#PWR018" H 2950 4150 50  0001 C CNN
 F 1 "GND" H 2950 4250 50  0000 C CNN
 F 2 "" H 2950 4400 60  0000 C CNN
@@
 $EndComp
 $Comp
-L GND #PWR20
+L GND #PWR019
 U 1 1 551C0D06
 P 3250 4400
-F 0 "#PWR20" H 3250 4150 50  0001 C CNN
+F 0 "#PWR019" H 3250 4150 50  0001 C CNN
 F 1 "GND" H 3250 4250 50  0000 C CNN
 F 2 "" H 3250 4400 60  0000 C CNN
@@
 F 0 "C13" H 3025 5150 50  0000 L CNN
 F 1 "15pF" H 3025 4950 50  0000 L CNN
-F 2 "Capacitors_SMD:C_0402" H 3038 4900 30  0001 C CNN
+F 2 "Capacitors_SMD:C_0603" H 3038 4900 30  0001 C CNN
 F 3 "" H 3000 5050 60  0000 C CNN
 	1    3000 5050
@@
 F 0 "C14" H 3025 5800 50  0000 L CNN
 F 1 "15pF" H 3025 5600 50  0000 L CNN
-F 2 "Capacitors_SMD:C_0402" H 3038 5550 30  0001 C CNN
+F 2 "Capacitors_SMD:C_0603" H 3038 5550 30  0001 C CNN
 F 3 "" H 3000 5700 60  0000 C CNN
 	1    3000 5700
@@
 $EndComp
 $Comp
-L GND #PWR16
+L GND #PWR020
 U 1 1 551C1217
 P 2350 5800
-F 0 "#PWR16" H 2350 5550 50  0001 C CNN
+F 0 "#PWR020" H 2350 5550 50  0001 C CNN
 F 1 "GND" H 2350 5650 50  0000 C CNN
 F 2 "" H 2350 5800 60  0000 C CNN
@@
 $EndComp
 $Comp
-L GND #PWR21
+L GND #PWR021
 U 1 1 551C134D
 P 4700 4500
-F 0 "#PWR21" H 4700 4250 50  0001 C CNN
+F 0 "#PWR021" H 4700 4250 50  0001 C CNN
 F 1 "GND" H 4700 4350 50  0000 C CNN
 F 2 "" H 4700 4500 60  0000 C CNN
@@
 $EndComp
 $Comp
-L GND #PWR23
+L GND #PWR022
 U 1 1 551C13DC
 P 5050 5400
-F 0 "#PWR23" H 5050 5150 50  0001 C CNN
+F 0 "#PWR022" H 5050 5150 50  0001 C CNN
 F 1 "GND" H 5050 5250 50  0000 C CNN
 F 2 "" H 5050 5400 60  0000 C CNN
@@
 F 0 "C16" H 5075 5350 50  0000 L CNN
 F 1 "100nF" H 5075 5150 50  0000 L CNN
-F 2 "Capacitors_SMD:C_0402" H 5088 5100 30  0001 C CNN
+F 2 "Capacitors_SMD:C_0603" H 5088 5100 30  0001 C CNN
 F 3 "" H 5050 5250 60  0000 C CNN
 	1    5050 5250
@@
 $EndComp
 $Comp
-L GND #PWR24
+L GND #PWR023
 U 1 1 551C159D
 P 5150 2950
-F 0 "#PWR24" H 5150 2700 50  0001 C CNN
+F 0 "#PWR023" H 5150 2700 50  0001 C CNN
 F 1 "GND" H 5150 2800 50  0000 C CNN
 F 2 "" H 5150 2950 60  0000 C CNN
@@
 F 0 "C17" H 7025 1350 50  0000 L CNN
 F 1 "12pF" H 7025 1150 50  0000 L CNN
-F 2 "Capacitors_SMD:C_0402" H 7038 1100 30  0001 C CNN
+F 2 "Capacitors_SMD:C_0603" H 7038 1100 30  0001 C CNN
 F 3 "" H 7000 1250 60  0000 C CNN
 	1    7000 1250
@@
 F 0 "C18" H 7025 2050 50  0000 L CNN
 F 1 "12pF" H 7025 1850 50  0000 L CNN
-F 2 "Capacitors_SMD:C_0402" H 7038 1800 30  0001 C CNN
+F 2 "Capacitors_SMD:C_0603" H 7038 1800 30  0001 C CNN
 F 3 "" H 7000 1950 60  0000 C CNN
 	1    7000 1950
@@
 $EndComp
 $Comp
-L GND #PWR29
+L GND #PWR024
 U 1 1 551C18D0
 P 7550 2150
-F 0 "#PWR29" H 7550 1900 50  0001 C CNN
+F 0 "#PWR024" H 7550 1900 50  0001 C CNN
 F 1 "GND" H 7550 2000 50  0000 C CNN
 F 2 "" H 7550 2150 60  0000 C CNN
@@
 $EndComp
 $Comp
-L R R5
+L R R6
 U 1 1 551C1DE2
 P 6450 2900
-F 0 "R5" V 6530 2900 50  0000 C CNN
+F 0 "R6" V 6530 2900 50  0000 C CNN
 F 1 "22k" V 6450 2900 50  0000 C CNN
-F 2 "Resistors_SMD:R_0402" V 6380 2900 30  0001 C CNN
+F 2 "Resistors_SMD:R_0603" V 6380 2900 30  0001 C CNN
 F 3 "" H 6450 2900 30  0000 C CNN
 	1    6450 2900
@@
 $EndComp
 $Comp
-L GND #PWR28
+L GND #PWR025
 U 1 1 551C1EC5
 P 7200 3000
-F 0 "#PWR28" H 7200 2750 50  0001 C CNN
+F 0 "#PWR025" H 7200 2750 50  0001 C CNN
 F 1 "GND" H 7200 2850 50  0000 C CNN
 F 2 "" H 7200 3000 60  0000 C CNN
@@
 F 0 "C19" H 7225 2850 50  0000 L CNN
 F 1 "1.0nF" H 7225 2650 50  0000 L CNN
-F 2 "Capacitors_SMD:C_0402" H 7238 2600 30  0001 C CNN
+F 2 "Capacitors_SMD:C_0603" H 7238 2600 30  0001 C CNN
 F 3 "" H 7200 2750 60  0000 C CNN
 	1    7200 2750
@@
 NoConn ~ 5900 4800
 $Comp
-L GND #PWR26
+L GND #PWR026
 U 1 1 551C247D
 P 6550 4450
-F 0 "#PWR26" H 6550 4200 50  0001 C CNN
+F 0 "#PWR026" H 6550 4200 50  0001 C CNN
 F 1 "GND" H 6550 4300 50  0000 C CNN
 F 2 "" H 6550 4450 60  0000 C CNN
@@
 $EndComp
 $Comp
-L GND #PWR30
+L GND #PWR027
 U 1 1 551C26C3
 P 8200 5100
-F 0 "#PWR30" H 8200 4850 50  0001 C CNN
+F 0 "#PWR027" H 8200 4850 50  0001 C CNN
 F 1 "GND" H 8200 4950 50  0000 C CNN
 F 2 "" H 8200 5100 60  0000 C CNN
@@
 $EndComp
 $Comp
-L GND #PWR31
+L GND #PWR028
 U 1 1 551C26F1
 P 8500 5100
-F 0 "#PWR31" H 8500 4850 50  0001 C CNN
+F 0 "#PWR028" H 8500 4850 50  0001 C CNN
 F 1 "GND" H 8500 4950 50  0000 C CNN
 F 2 "" H 8500 5100 60  0000 C CNN
@@
 F 0 "C20" H 8225 5050 50  0000 L CNN
 F 1 "2.2nF" H 8225 4850 50  0000 L CNN
-F 2 "Capacitors_SMD:C_0402" H 8238 4800 30  0001 C CNN
+F 2 "Capacitors_SMD:C_0603" H 8238 4800 30  0001 C CNN
 F 3 "" H 8200 4950 60  0000 C CNN
 	1    8200 4950
@@
 F 0 "C21" H 8525 5050 50  0000 L CNN
 F 1 "NC" H 8525 4850 50  0000 L CNN
-F 2 "Capacitors_SMD:C_0402" H 8538 4800 30  0001 C CNN
+F 2 "Capacitors_SMD:C_0603" H 8538 4800 30  0001 C CNN
 F 3 "" H 8500 4950 60  0000 C CNN
 	1    8500 4950
@@
 F 0 "L1" V 7450 4050 50  0000 C CNN
 F 1 "8.2nH" V 7600 4050 50  0000 C CNN
-F 2 "Capacitors_SMD:C_0402" H 7500 4050 60  0001 C CNN
+F 2 "Capacitors_SMD:C_0603" H 7500 4050 60  0001 C CNN
 F 3 "" H 7500 4050 60  0000 C CNN
 	1    7500 4050
@@
 F 0 "L2" V 8050 3750 50  0000 C CNN
 F 1 "3.9nH" V 8200 3750 50  0000 C CNN
-F 2 "" H 8100 3750 60  0001 C CNN
+F 2 "Capacitors_SMD:C_0603" H 8100 3750 60  0001 C CNN
 F 3 "" H 8100 3750 60  0000 C CNN
 	1    8100 3750
@@
 F 0 "L3" V 8050 4350 50  0000 C CNN
 F 1 "5.6nH" V 8200 4350 50  0000 C CNN
-F 2 "Capacitors_SMD:C_0402" H 8100 4350 60  0001 C CNN
+F 2 "Capacitors_SMD:C_0603" H 8100 4350 60  0001 C CNN
 F 3 "" H 8100 4350 60  0000 C CNN
 	1    8100 4350
@@
 F 0 "C22" H 9025 3850 50  0000 L CNN
 F 1 "1.8pF" H 9025 3650 50  0000 L CNN
-F 2 "Capacitors_SMD:C_0402" H 9038 3600 30  0001 C CNN
+F 2 "Capacitors_SMD:C_0603" H 9038 3600 30  0001 C CNN
 F 3 "" H 9000 3750 60  0000 C CNN
 	1    9000 3750
@@
 F 0 "C23" H 9725 4200 50  0000 L CNN
 F 1 "1.2pF" H 9725 4000 50  0000 L CNN
-F 2 "Capacitors_SMD:C_0402" H 9738 3950 30  0001 C CNN
+F 2 "Capacitors_SMD:C_0603" H 9738 3950 30  0001 C CNN
 F 3 "" H 9700 4100 60  0000 C CNN
 	1    9700 4100
@@
 $EndComp
 $Comp
-L GND #PWR32
+L GND #PWR029
 U 1 1 551C3732
 P 9700 4400
-F 0 "#PWR32" H 9700 4150 50  0001 C CNN
+F 0 "#PWR029" H 9700 4150 50  0001 C CNN
 F 1 "GND" H 9700 4250 50  0000 C CNN
 F 2 "" H 9700 4400 60  0000 C CNN
@@
 	5800 1950 6850 1950
 $Comp
-L +3V #PWR17
+L +3V #PWR030
 U 1 1 55282769
 P 2650 3550
-F 0 "#PWR17" H 2650 3450 60  0001 C CNN
+F 0 "#PWR030" H 2650 3450 60  0001 C CNN
 F 1 "+3V" H 2500 3700 60  0000 C CNN
 F 2 "" H 2650 3550 60  0000 C CNN
@@
 $EndComp
 $Comp
-L +3V #PWR22
+L +3V #PWR031
 U 1 1 5528286C
 P 5050 4950
-F 0 "#PWR22" H 5050 4850 60  0001 C CNN
+F 0 "#PWR031" H 5050 4850 60  0001 C CNN
 F 1 "+3V" H 4900 5100 60  0000 C CNN
 F 2 "" H 5050 4950 60  0000 C CNN
@@
 $EndComp
 $Comp
-L +3V #PWR25
+L +3V #PWR032
 U 1 1 552829BF
 P 5600 2900
-F 0 "#PWR25" H 5600 2800 60  0001 C CNN
+F 0 "#PWR032" H 5600 2800 60  0001 C CNN
 F 1 "+3V" H 5450 3050 60  0000 C CNN
 F 2 "" H 5600 2900 60  0000 C CNN
@@
 $EndComp
 $Comp
-L +3V #PWR27
+L +3V #PWR033
 U 1 1 55282B5E
 P 7200 2550
-F 0 "#PWR27" H 7200 2450 60  0001 C CNN
+F 0 "#PWR033" H 7200 2450 60  0001 C CNN
 F 1 "+3V" H 7050 2700 60  0000 C CNN
 F 2 "" H 7200 2550 60  0000 C CNN

Commit message: pre major restructuring commit
Parts:
- removed C21: NC, Capacitors_SMD:C_0603, symbol C
- removed C22: 1.8pF, Capacitors_SMD:C_0603, symbol C
- removed C23: 1.2pF, Capacitors_SMD:C_0603, symbol C
- removed L1: 8.2nH, Capacitors_SMD:C_0603, symbol INDUCTOR
- removed L2: 3.9nH, Capacitors_SMD:C_0603, symbol INDUCTOR
- removed L3: 5.6nH, Capacitors_SMD:C_0603, symbol INDUCTOR
- added A1: 2450AT18A100, aero:2450AT18A100, symbol 2450AT18A100
- added U3: 2450BM14A0002, aero:2450BM14A0002, symbol 2450BM14A0002
- C11, C12, C13, C14, C15, C16, C17, C18, C19, C20: footprint Capacitors_SMD:C_0603 -> Capacitors_SMD:C_0402
- R5: renamed from R6; footprint Resistors_SMD:R_0603 -> Resistors_SMD:R_0402
- U2: footprint Housings_DFN_QFN:QFN-32-1EP_5x5mm_Pitch0.5mm -> aero:QFN-32-1EP_5x5mm_Pitch0.5mm
- Y3: footprint aero:FC-135R -> (none)
- Y4: footprint aero:crystal_SMD_3225 -> (none)
Connections:
- net GND: now also U3.2 (GND)
- net at C20.1, U2.20 (VDD_PA): now also U3.5 (DC)
- net at U2.21 (ANT1): now also U3.4 (Bal2)
- net at U2.22 (ANT2): now also U3.3 (Bal1)
- new net: A1.1 (Feed), U3.1 (Unbal)
Other:
- moved on the sheet: C20

Commit message: committing before shit starts breaking (pcbnew)
Parts:
- Y3: footprint (none) -> aero:Crystal_32768_FC-135R
Changed lines of the file:
@@
 F 0 "Y3" H 3600 5500 50  0000 C CNN
 F 1 "32.768KHz" H 3600 5200 50  0000 C CNN
-F 2 "" H 3600 5350 60  0001 C CNN
+F 2 "aero:Crystal_32768_FC-135R" H 3600 5350 60  0001 C CNN
 F 3 "" H 3600 5350 60  0000 C CNN
 	1    3600 5350

Commit message: more progress on new layout
Parts:
- Y3: renamed from Y4; footprint (none) -> aero:Crystal_TSX_3225
- renumbered C12 to C10, C13 to C11, C14 to C12, C15 to C13, C16 to C14, C17 to C15, C18 to C16, C19 to C17, C20 to C18, C11 to C9, R5 to R4, Y3 to Y2
Changed lines of the file:
@@
 $EndComp
 $Comp
-L C C11
+L C C9
 U 1 1 551C0AC5
 P 2650 4200
-F 0 "C11" H 2675 4300 50  0000 L CNN
+F 0 "C9" H 2675 4300 50  0000 L CNN
 F 1 "100nF" H 2675 4100 50  0000 L CNN
 F 2 "Capacitors_SMD:C_0402" H 2688 4050 30  0001 C CNN
@@
 $EndComp
 $Comp
-L C C12
+L C C10
 U 1 1 551C0AEF
 P 2950 4200
-F 0 "C12" H 2975 4300 50  0000 L CNN
+F 0 "C10" H 2975 4300 50  0000 L CNN
 F 1 "100nF" H 2975 4100 50  0000 L CNN
 F 2 "Capacitors_SMD:C_0402" H 2988 4050 30  0001 C CNN
@@
 $EndComp
 $Comp
-L C C15
+L C C13
 U 1 1 551C0B13
 P 3250 4200
-F 0 "C15" H 3275 4300 50  0000 L CNN
+F 0 "C13" H 3275 4300 50  0000 L CNN
 F 1 "33nF" H 3275 4100 50  0000 L CNN
 F 2 "Capacitors_SMD:C_0402" H 3288 4050 30  0001 C CNN
@@
 $EndComp
 $Comp
-L Crystal Y3
+L Crystal Y2
 U 1 1 551C0F7F
 P 3600 5350
-F 0 "Y3" H 3600 5500 50  0000 C CNN
+F 0 "Y2" H 3600 5500 50  0000 C CNN
 F 1 "32.768KHz" H 3600 5200 50  0000 C CNN
 F 2 "aero:Crystal_32768_FC-135R" H 3600 5350 60  0001 C CNN
@@
 $EndComp
 $Comp
-L C C13
+L C C11
 U 1 1 551C1027
 P 3000 5050
-F 0 "C13" H 3025 5150 50  0000 L CNN
+F 0 "C11" H 3025 5150 50  0000 L CNN
 F 1 "15pF" H 3025 4950 50  0000 L CNN
 F 2 "Capacitors_SMD:C_0402" H 3038 4900 30  0001 C CNN
@@
 $EndComp
 $Comp
-L C C14
+L C C12
 U 1 1 551C108E
 P 3000 5700
-F 0 "C14" H 3025 5800 50  0000 L CNN
+F 0 "C12" H 3025 5800 50  0000 L CNN
 F 1 "15pF" H 3025 5600 50  0000 L CNN
 F 2 "Capacitors_SMD:C_0402" H 3038 5550 30  0001 C CNN
@@
 $EndComp
 $Comp
-L C C16
+L C C14
 U 1 1 551C140C
 P 5050 5250
-F 0 "C16" H 5075 5350 50  0000 L CNN
+F 0 "C14" H 5075 5350 50  0000 L CNN
 F 1 "100nF" H 5075 5150 50  0000 L CNN
 F 2 "Capacitors_SMD:C_0402" H 5088 5100 30  0001 C CNN
@@
 $EndComp
 $Comp
-L Crystal Y4
+L Crystal Y3
 U 1 1 551C1703
 P 6450 1600
-F 0 "Y4" H 6450 1750 50  0000 C CNN
+F 0 "Y3" H 6450 1750 50  0000 C CNN
 F 1 "16MHz" H 6450 1450 50  0000 C CNN
-F 2 "" H 6450 1600 60  0001 C CNN
+F 2 "aero:Crystal_TSX_3225" H 6450 1600 60  0001 C CNN
 F 3 "" H 6450 1600 60  0000 C CNN
 	1    6450 1600
@@
 $EndComp
 $Comp
-L C C17
+L C C15
 U 1 1 551C17DD
 P 7000 1250
-F 0 "C17" H 7025 1350 50  0000 L CNN
+F 0 "C15" H 7025 1350 50  0000 L CNN
 F 1 "12pF" H 7025 1150 50  0000 L CNN
 F 2 "Capacitors_SMD:C_0402" H 7038 1100 30  0001 C CNN
@@
 $EndComp
 $Comp
-L C C18
+L C C16
 U 1 1 551C1811
 P 7000 1950
-F 0 "C18" H 7025 2050 50  0000 L CNN
+F 0 "C16" H 7025 2050 50  0000 L CNN
 F 1 "12pF" H 7025 1850 50  0000 L CNN
 F 2 "Capacitors_SMD:C_0402" H 7038 1800 30  0001 C CNN
@@
 $EndComp
 $Comp
-L R R5
+L R R4
 U 1 1 551C1DE2
 P 6450 2900
-F 0 "R5" V 6530 2900 50  0000 C CNN
+F 0 "R4" V 6530 2900 50  0000 C CNN
 F 1 "22k" V 6450 2900 50  0000 C CNN
 F 2 "Resistors_SMD:R_0402" V 6380 2900 30  0001 C CNN
@@
 $EndComp
 $Comp
-L C C19
+L C C17
 U 1 1 551C2016
 P 7200 2750
-F 0 "C19" H 7225 2850 50  0000 L CNN
+F 0 "C17" H 7225 2850 50  0000 L CNN
 F 1 "1.0nF" H 7225 2650 50  0000 L CNN
 F 2 "Capacitors_SMD:C_0402" H 7238 2600 30  0001 C CNN
@@
 $EndComp
 $Comp
-L C C20
+L C C18
 U 1 1 551C277F
 P 8050 4750
-F 0 "C20" H 8075 4850 50  0000 L CNN
+F 0 "C18" H 8075 4850 50  0000 L CNN
 F 1 "2.2nF" H 8075 4650 50  0000 L CNN
 F 2 "Capacitors_SMD:C_0402" H 8088 4600 30  0001 C CNN
