File: hardware/pcb/aero.sch (KiCad schematic (older format))
At the start: 9 parts

Commit message: schematic updates
Connections:
- net GND: now also R?.2; no longer R?.1
- net warn/PIEZO_EN: now also U?.42 (PB6/I2C1_SCL/TIM4_CH1/USART1_TX)
- net warn/PIEZO_OUT: now also U?.43 (PB7/I2C1_SDA/TIM4_CH2/USART1_RX/PVD_IN)
- net warn/STATUS_LED: now also U?.22 (PB11/I2C2_SDA/USART3_RX/TIM2_CH4)
- net warn/WARN_LED_EN: now also U?.46 (PB9/TIM4_CH4/I2C1_SDA/TIM11_CH1)
- net warn/WARN_LED_SELECT: now also U?.45 (PB8/TIM4_CH3/I2C1_SCL/TIM10_CH1)
- net NRF8001_ENABLE: now reaches U?.21 (PB10/I2C2_SCL/USART3_TX/TIM2_CH3)
- net at D?.1 (K): now also R?.1; no longer R?.2
Other:
- moved on the sheet: D?, R?

Commit message: schematic updates
Parts:
- added 10k, R? (x2): R, symbol R
- added C? (x4): C, symbol C
- added Y? (x2): Crystal_Small, symbol Crystal_Small
Connections:
- net labels added: SWO, ~NRST
- wire segments 119 -> 167
Other:
- moved on the sheet: D?, J?, R?

Commit message: Added some testpoints
Parts:
- removed Y?: Crystal_Small, symbol Crystal_Small
- added TP? (x10): Test_Point, symbol Test_Point
- added Y?: Crystal, symbol Crystal
- Y?: value Crystal_Small -> Crystal; symbol Crystal_Small -> Crystal
Connections:
- wire segments 167 -> 151
Other:
- moved on the sheet: C?, R?

Commit message: schematic nearing completion
Parts:
- removed R?: R, symbol R
- added R?: 0, symbol R
- C? (x4): value C -> 100n
- C?: value C -> 1u
- C? (x2): value C -> 15p
- R?: value R -> 220
- Y?: footprint (none) -> aero:FC-135R
Connections:
- net GND: now also 10k.2
- net at U?.4 (PC15/OSC32_OUT): now also R?.2
- net at C?.1, Y?.1: now also R?.1
- net warn/WARN_LED_EN renamed warn/WARN_LED_B
- net warn/WARN_LED_SELECT renamed warn/WARN_LED_A
Other:
- note added: "HSE"
- note added: "LSE"
- note added: "NOT FITTED"
Changed lines of the file:
@@
 P 700 7100
 F 0 "C?" H 725 7200 50  0000 L CNN
-F 1 "C" H 725 7000 50  0000 L CNN
+F 1 "100n" H 725 7000 50  0000 L CNN
 F 2 "" H 738 6950 30  0000 C CNN
 F 3 "" H 700 7100 60  0000 C CNN
@@
 P 1000 7100
 F 0 "C?" H 1025 7200 50  0000 L CNN
-F 1 "C" H 1025 7000 50  0000 L CNN
+F 1 "100n" H 1025 7000 50  0000 L CNN
 F 2 "" H 1038 6950 30  0000 C CNN
 F 3 "" H 1000 7100 60  0000 C CNN
@@
 P 1300 7100
 F 0 "C?" H 1325 7200 50  0000 L CNN
-F 1 "C" H 1325 7000 50  0000 L CNN
+F 1 "100n" H 1325 7000 50  0000 L CNN
 F 2 "" H 1338 6950 30  0000 C CNN
 F 3 "" H 1300 7100 60  0000 C CNN
@@
 P 1600 7100
 F 0 "C?" H 1625 7200 50  0000 L CNN
-F 1 "C" H 1625 7000 50  0000 L CNN
+F 1 "100n" H 1625 7000 50  0000 L CNN
 F 2 "" H 1638 6950 30  0000 C CNN
 F 3 "" H 1600 7100 60  0000 C CNN
@@
 P 1900 7100
 F 0 "C?" H 1925 7200 50  0000 L CNN
-F 1 "C" H 1925 7000 50  0000 L CNN
+F 1 "1u" H 1925 7000 50  0000 L CNN
 F 2 "" H 1938 6950 30  0000 C CNN
 F 3 "" H 1900 7100 60  0000 C CNN
@@
 F2 "PIEZO_EN" I R 1650 3000 60
 F3 "PIEZO_OUT" I R 1650 3100 60
-F4 "WARN_LED_SELECT" I R 1650 3200 60
-F5 "WARN_LED_EN" I R 1650 3300 60
-F6 "STATUS_LED" I R 1650 3400 60
+F4 "STATUS_LED" I R 1650 3400 60
+F5 "WARN_LED_A" I R 1650 3200 60
+F6 "WARN_LED_B" I R 1650 3300 60
 $EndSheet
 Text GLabel 3450 5300 0    60   Input ~ 0
@@
 P 2850 850
 F 0 "C?" H 2875 950 50  0000 L CNN
-F 1 "C" H 2875 750 50  0000 L CNN
+F 1 "15p" H 2875 750 50  0000 L CNN
 F 2 "" H 2888 700 30  0000 C CNN
 F 3 "" H 2850 850 60  0000 C CNN
@@
 P 3750 850
 F 0 "C?" H 3775 950 50  0000 L CNN
-F 1 "C" H 3775 750 50  0000 L CNN
+F 1 "15p" H 3775 750 50  0000 L CNN
 F 2 "" H 3788 700 30  0000 C CNN
 F 3 "" H 3750 850 60  0000 C CNN
@@
 F 3 "" H 4050 950 60  0000 C CNN
 	1    4050 950
-	1    0    0    -1
-$EndComp
-$Comp
-L R R?
-U 1 1 553A0C35
-P 3100 1150
-F 0 "R?" V 3180 1150 50  0000 C CNN
-F 1 "R" V 3100 1150 50  0000 C CNN
-F 2 "" V 3030 1150 30  0000 C CNN
-F 3 "" H 3100 1150 30  0000 C CNN
-	1    3100 1150
 	1    0    0    -1
 $EndComp
@@
 P 5200 1200
 F 0 "R?" V 5280 1200 50  0000 C CNN
-F 1 "R" V 5200 1200 50  0000 C CNN
+F 1 "220" V 5200 1200 50  0000 C CNN
 F 2 "" V 5130 1200 30  0000 C CNN
 F 3 "" H 5200 1200 30  0000 C CNN
@@
 Wire Wire Line
 	2500 850  2500 950
-Wire Wire Line
-	3100 1000 3100 850
 Connection ~ 3100 850
-Wire Wire Line
-	3100 1300 3100 3950
 Wire Wire Line
 	3100 3950 4250 3950
@@
 F 0 "Y?" H 3300 1000 50  0000 C CNN
 F 1 "Crystal" H 3300 700 50  0000 C CNN
-F 2 "" H 3300 850 60  0000 C CNN
+F 2 "aero:FC-135R" H 3700 1000 60  0000 C CNN
 F 3 "" H 3300 850 60  0000 C CNN
 	1    3300 850
@@
 Wire Wire Line
 	3450 850  3600 850
+Text Notes 3050 650  0    60   ~ 0
+LSE
+Text Notes 5100 750  0    60   ~ 0
+HSE
+$Comp
+L GND #PWR?
+U 1 1 553AC8AD
+P 3800 3250
+F 0 "#PWR?" H 3800 3000 50  0001 C CNN
+F 1 "GND" H 3800 3100 50  0000 C CNN
+F 2 "" H 3800 3250 60  0000 C CNN
+F 3 "" H 3800 3250 60  0000 C CNN
+	1    3800 3250
+	1    0    0    -1
+$EndComp
+Wire Wire Line
+	3800 3200 3800 3250
+Wire Notes Line
+	4450 500  4450 1550
+Wire Notes Line
+	4450 1550 6350 1550
+Wire Notes Line
+	6350 1550 6350 500
+Wire Notes Line
+	6350 500  4450 500
+Text Notes 5800 600  0    60   ~ 0
+NOT FITTED
+$Comp
+L R R?
+U 1 1 553B1F5F
+P 3100 1200
+F 0 "R?" V 3180 1200 50  0000 C CNN
+F 1 "0" V 3100 1200 50  0000 C CNN
+F 2 "" V 3030 1200 30  0000 C CNN
+F 3 "" H 3100 1200 30  0000 C CNN
+	1    3100 1200
+	1    0    0    -1
+$EndComp
+Wire Wire Line
+	3100 1050 3100 850
+Wire Wire Line
+	3100 1350 3100 3950
 $EndSCHEMATC

Commit message: schematic updates
Connections:
- no-connect marks 2 -> 1
Changed lines of the file:
@@
 Text GLabel 9950 4050 0    60   Input ~ 0
 NRF8001_ENABLE
-NoConn ~ 1550 5200
 Text GLabel 4100 3050 0    60   Input ~ 0
 ~NRST
@@
 Wire Wire Line
 	3100 1350 3100 3950
+Text GLabel 1600 5200 2    60   Input ~ 0
+ACC_INT
+Wire Wire Line
+	1600 5200 1550 5200
 $EndSCHEMATC

Commit message: more changes
Parts:
- added C8: 10nF, symbol C
- added SW1: SW_PUSH, symbol SW_PUSH
- C1, C2, C3, C4: renamed from C?; value 100n -> 100nF
- C5: renamed from C?; value 1u -> 1uF
- C6, C7: renamed from C?; value 15p -> 9pF
- R2: renamed from 10k; value R -> 10k
- gave numbers to parts that had none: 20
Connections:
- net ACC_INT: now also U1.40 (PB4/NJRST/TIM3_CH1/SPI1_MISO/COMP2_INP)
- net GND: now also C8.2, SW1.2
- net ~NRST: now also C8.1, SW1.1
- net ~PG: now reaches U1.19 (PB1/ADC_IN9/TIM3_CH4/COMP1_INP/VREF_OUT)
- no-connect marks 1 -> 7

Commit message: mega commit
Parts:
- added R4: 1.5k, Resistors_SMD:R_0603, symbol R
- C1, C2, C3, C4, C5, C6, C7, C8: footprint (none) -> Capacitors_SMD:C_0603
- C10, C9: value C -> 15pF; footprint (none) -> Capacitors_SMD:C_0603
- D1: footprint (none) -> LEDs:LED-0805
- J1: footprint (none) -> aero:FTSH-105-01
- R1, R2, R3: footprint (none) -> Resistors_SMD:R_0603
- R5: renamed from R4; footprint (none) -> Resistors_SMD:R_0603
- SW1: footprint (none) -> aero:B3U-1000P
- TP1, TP10, TP2, TP3, TP4, TP5, TP6, TP7, TP8, TP9: footprint (none) -> aero:TP_0603
- Y2: footprint (none) -> aero:Murata_CSTCE-G_Oscillator
Connections:
- net +3V3: now also R4.1
- net power/USB_D+: now also R4.2
