File: hardware/pcb/aero.sch (KiCad schematic (older format))
At the start: 31 parts, among them J1 CORTEX_DBG_CONN, SW1 SW_PUSH, U1 STM32L151C8, Y1 Crystal, Y2 Crystal

Commit message: pre major restructuring commit
Parts:
- removed C10, C9: 15pF, Capacitors_SMD:C_0603, symbol C
- removed D1: LED, LEDs:LED-0805, symbol LED
- removed R3: 220, Resistors_SMD:R_0603, symbol R
- removed R5: 1.5k, Resistors_SMD:R_0603, symbol R
- removed TP1, TP2, TP3, TP4: Test_Point, aero:TP_0603, symbol Test_Point
- removed Y2: Crystal, aero:Murata_CSTCE-G_Oscillator, symbol Crystal
- C1, C2, C3, C4, C5, C6, C7, C8: footprint Capacitors_SMD:C_0603 -> Capacitors_SMD:C_0402
- J1: footprint aero:FTSH-105-01 -> aero:TC2050-IDC-NL
- R1, R2, R4: footprint Resistors_SMD:R_0603 -> Resistors_SMD:R_0402
- Y1: footprint aero:FC-135R -> aero:crystal_SMD_3225
- renumbered TP5 to TP1, TP6 to TP2, TP7 to TP3, TP8 to TP4, TP9 to TP5, TP10 to TP6
Connections:
- net ACC_INT is gone; now on net warn/PIEZO_EN: U1.40 (PB4/NJRST/TIM3_CH1/SPI1_MISO/COMP2_INP)
- net ACC_SEL is gone; now on net ~PG: U1.30 (USART1_TX/PA9)
- net warn/PIEZO_EN: no longer U1.42 (PB6/I2C1_SCL/TIM4_CH1/USART1_TX)
- net warn/PIEZO_OUT: now also U1.41 (PB5/I2C1_SMBDAI/TIM3_CH2/SPI1_MOSI/COMP2_INP); no longer U1.43 (PB7/I2C1_SDA/TIM4_CH2/USART1_RX/PVD_IN)
- net ~PG: no longer U1.19 (PB1/ADC_IN9/TIM3_CH4/COMP1_INP/VREF_OUT)
- net bmx055/ACC_SEL: now reaches U1.18 (PB0/ADC_IN8/TIM3_CH3/COMP1_INP/VREF_OUT)
- net GPS/TIMEPULSE: now reaches U1.2 (PC13/TAMPER_RTC)
- net bmx055/MAG_SEL: now reaches U1.20 (PB2/BOOT1)
- net GPS/RESET: now reaches U1.5 (PH0/OSC_IN)
- net GYRO_SEL renamed ~CHG
- net MAG_SEL renamed GPS_INT
- new net GPS/RxD: U1.42 (PB6/I2C1_SCL/TIM4_CH1/USART1_TX)
- new net GPS/TxD: U1.43 (PB7/I2C1_SDA/TIM4_CH2/USART1_RX/PVD_IN)
- new net bmx055/GYRO_SEL: U1.19 (PB1/ADC_IN9/TIM3_CH4/COMP1_INP/VREF_OUT)
Other:
- note added: "Alti"
- note removed: "HSE"
- note removed: "NOT FITTED"

Commit message: committing before shit starts breaking (pcbnew)
Connections:
- net GPS/EXT_INT: now reaches U1.6 (PH1/OSC_OUT)
- net GPS_INT: no longer names the net of U1.29 (USART1_CK/MCO/PA8)
Changed lines of the file:
@@
 	10200 5750 9700 5750
 Wire Wire Line
-	9700 4950 9700 5750
-Wire Wire Line
-	8500 4950 9700 4950
+	9700 5750 9700 4950
+Wire Wire Line
+	9700 4950 8500 4950
 Wire Wire Line
 	8500 4950 8500 4400
@@
 	2975 4700 4250 4700
 $Sheet
-S 650  700  875  650
+S 675  700  900  800
 U 55B6C26A
 F0 "GPS" 60
 F1 "GPS.sch" 60
-F2 "TIMEPULSE" I R 1525 1325 60
-F3 "TxD" I R 1525 875 60
-F4 "RxD" I R 1525 800 60
-F5 "SDA" I R 1525 975 60
-F6 "SCL" I R 1525 1050 60
-F7 "EXT_INT" I R 1525 1250 60
-F8 "RESET" I R 1525 1150 60
+F2 "TIMEPULSE" I R 1575 1125 60
+F3 "TxD" I R 1575 1425 60
+F4 "RxD" I R 1575 1350 60
+F5 "SDA" I R 1575 775 60
+F6 "SCL" I R 1575 850 60
+F7 "EXT_INT" I R 1575 1050 60
+F8 "RESET" I R 1575 975 60
 $EndSheet
-Wire Wire Line
-	1525 800  2400 800
-Wire Wire Line
-	2400 800  2400 1950
-Wire Wire Line
-	2400 1950 3350 1950
-Wire Wire Line
-	3350 1950 3350 4900
-Wire Wire Line
-	3350 4900 4250 4900
-Wire Wire Line
-	1525 875  2300 875
-Wire Wire Line
-	2300 875  2300 2025
-Wire Wire Line
-	2300 2025 3275 2025
-Wire Wire Line
-	3275 2025 3275 5000
-Wire Wire Line
-	3275 5000 4250 5000
-NoConn ~ 1525 975
-NoConn ~ 1525 1050
-Wire Wire Line
-	1525 1150 2175 1150
-Wire Wire Line
-	2175 1150 2175 2150
-Wire Wire Line
-	2175 2150 3200 2150
-Wire Wire Line
-	3200 2150 3200 3400
-Wire Wire Line
-	3200 3400 4250 3400
-Wire Wire Line
-	4250 3750 3050 3750
-Wire Wire Line
-	3050 3750 3050 2375
-Wire Wire Line
-	3050 2375 1725 2375
-Wire Wire Line
-	1725 2375 1725 1325
-Wire Wire Line
-	1725 1325 1525 1325
-NoConn ~ 4250 3550
-Text GLabel 1700 1250 2    60   Input ~ 0
-GPS_INT
-Text GLabel 7550 4000 2    60   Input ~ 0
-GPS_INT
-Wire Wire Line
-	7550 4000 7450 4000
-Wire Wire Line
-	1700 1250 1525 1250
+NoConn ~ 7450 4000
+NoConn ~ 1575 775
+NoConn ~ 1575 850
+Wire Wire Line
+	1575 975  2300 975
+Wire Wire Line
+	2300 975  2300 1600
+Wire Wire Line
+	2300 1600 3325 1600
+Wire Wire Line
+	3325 1600 3325 3400
+Wire Wire Line
+	3325 3400 4250 3400
+Wire Wire Line
+	1575 1050 2225 1050
+Wire Wire Line
+	2225 1050 2225 1675
+Wire Wire Line
+	2225 1675 3275 1675
+Wire Wire Line
+	3275 1675 3275 3550
+Wire Wire Line
+	3275 3550 4250 3550
+Wire Wire Line
+	1575 1125 2150 1125
+Wire Wire Line
+	2150 1125 2150 1775
+Wire Wire Line
+	2150 1775 3200 1775
+Wire Wire Line
+	3200 1775 3200 3750
+Wire Wire Line
+	3200 3750 4250 3750
+Wire Wire Line
+	4250 4900 3125 4900
+Wire Wire Line
+	3125 4900 3125 1850
+Wire Wire Line
+	3125 1850 2075 1850
+Wire Wire Line
+	2075 1850 2075 1350
+Wire Wire Line
+	2075 1350 1575 1350
+Wire Wire Line
+	4250 5000 3050 5000
+Wire Wire Line
+	3050 5000 3050 1925
+Wire Wire Line
+	3050 1925 1975 1925
+Wire Wire Line
+	1975 1925 1975 1425
+Wire Wire Line
+	1975 1425 1575 1425
 $EndSCHEMATC

Commit message: more progress on new layout
Parts:
- Y1: footprint aero:crystal_SMD_3225 -> aero:Crystal_32768_FC-135R
- renumbered R4 to R3
Changed lines of the file:
@@
 F 0 "Y1" H 3300 1000 50  0000 C CNN
 F 1 "Crystal" H 3300 700 50  0000 C CNN
-F 2 "aero:crystal_SMD_3225" H 3700 1000 60  0001 C CNN
+F 2 "aero:Crystal_32768_FC-135R" H 3700 1000 60  0001 C CNN
 F 3 "" H 3300 850 60  0000 C CNN
 	1    3300 850
@@
 $EndComp
 $Comp
-L R R4
+L R R3
 U 1 1 553FF368
 P 9100 4700
-F 0 "R4" V 9180 4700 50  0000 C CNN
+F 0 "R3" V 9180 4700 50  0000 C CNN
 F 1 "1.5k" V 9100 4700 50  0000 C CNN
 F 2 "Resistors_SMD:R_0402" V 9030 4700 30  0001 C CNN

Commit message: ver2 is nearing completion.
Connections:
- net GPS/RxD is gone; now on net ~CHG: U1.42 (PB6/I2C1_SCL/TIM4_CH1/USART1_TX)
- net GPS/TxD is gone; now on net ~PG: U1.43 (PB7/I2C1_SDA/TIM4_CH2/USART1_RX/PVD_IN)
- net GPS/RESET: now also U1.2 (PC13/TAMPER_RTC); no longer U1.5 (PH0/OSC_IN)
- net GPS/TIMEPULSE: now also U1.5 (PH0/OSC_IN); no longer U1.2 (PC13/TAMPER_RTC)
- net ~CHG: no longer U1.31 (USART1_RX/PA10)
- net ~PG: no longer U1.30 (USART1_TX/PA9)
- net MS5611_EN: now reaches U1.29 (USART1_CK/MCO/PA8)
- net ms5611/EN renamed BATT_SENSE
- new net GPS_RX: U1.30 (USART1_TX/PA9)
- new net GPS_TX: U1.31 (USART1_RX/PA10)
- no-connect marks 7 -> 6

Commit message: pre-net import
Connections:
- net at45db321e/~CS: now also U1.10 (WKUP/USART2_CTS/ADC_IN0/TIM2_CH1_ETR/COMP1_INP/PA0); no longer U1.11 (USART2_RTS/ADC_IN1/TIM2_CH2/COMP1_INP/PA1)
- net at45db321e/~RESET: now also U1.11 (USART2_RTS/ADC_IN1/TIM2_CH2/COMP1_INP/PA1); no longer U1.10 (WKUP/USART2_CTS/ADC_IN0/TIM2_CH1_ETR/COMP1_INP/PA0)
- net warn/PIEZO_EN: now also U1.45 (PB8/TIM4_CH3/I2C1_SCL/TIM10_CH1); no longer U1.40 (PB4/NJRST/TIM3_CH1/SPI1_MISO/COMP2_INP)
- net warn/PIEZO_OUT: now also U1.46 (PB9/TIM4_CH4/I2C1_SDA/TIM11_CH1); no longer U1.41 (PB5/I2C1_SMBDAI/TIM3_CH2/SPI1_MOSI/COMP2_INP)
- net warn/WARN_LED_A: now also U1.42 (PB6/I2C1_SCL/TIM4_CH1/USART1_TX); no longer U1.45 (PB8/TIM4_CH3/I2C1_SCL/TIM10_CH1)
- net warn/WARN_LED_B: now also U1.43 (PB7/I2C1_SDA/TIM4_CH2/USART1_RX/PVD_IN); no longer U1.46 (PB9/TIM4_CH4/I2C1_SDA/TIM11_CH1)
- net ~CHG: now also U1.40 (PB4/NJRST/TIM3_CH1/SPI1_MISO/COMP2_INP); no longer U1.42 (PB6/I2C1_SCL/TIM4_CH1/USART1_TX)
- net ~PG: now also U1.41 (PB5/I2C1_SMBDAI/TIM3_CH2/SPI1_MOSI/COMP2_INP); no longer U1.43 (PB7/I2C1_SDA/TIM4_CH2/USART1_RX/PVD_IN)
- net NRF8001_ENABLE renamed NRF8001_ACTIVE
Changed lines of the file:
@@
 $EndSheet
 Text GLabel 3450 5300 0    60   Input ~ 0
-NRF8001_ENABLE
+NRF8001_ACTIVE
 Text GLabel 9950 4050 0    60   Input ~ 0
-NRF8001_ENABLE
+NRF8001_ACTIVE
 Text GLabel 4100 3050 0    60   Input ~ 0
 ~NRST
@@
 NoConn ~ 10100 4150
 NoConn ~ 10100 4250
-Text GLabel 4150 5000 0    60   Input ~ 0
+Text GLabel 4025 4800 0    60   Input ~ 0
 ~PG
 Text GLabel 9975 5975 0    60   Input ~ 0
@@
 Text Notes 7375 7500 0    60   ~ 0
 Alti
-Text GLabel 4175 4900 0    60   Input ~ 0
+Text GLabel 4050 4700 0    60   Input ~ 0
 ~CHG
 Text GLabel 10000 5850 0    60   Input ~ 0
@@
 	9200 2700 10100 2700
 Wire Wire Line
-	10100 2800 9300 2800
-Wire Wire Line
-	9300 2800 9300 3300
-Wire Wire Line
-	9300 3300 7450 3300
-Wire Wire Line
-	10100 2900 9400 2900
-Wire Wire Line
-	9400 2900 9400 3200
-Wire Wire Line
-	9400 3200 7450 3200
+	9275 2800 9275 3200
+Wire Wire Line
+	9275 3200 7450 3200
 Wire Wire Line
 	9100 2600 10100 2600
@@
 	3450 5300 4250 5300
 Wire Wire Line
-	2650 5200 4250 5200
-Wire Wire Line
-	2650 5200 2650 3300
-Wire Wire Line
 	2650 3300 1650 3300
 Wire Wire Line
 	1650 3200 2750 3200
-Wire Wire Line
-	2750 3200 2750 5100
-Wire Wire Line
-	2750 5100 4250 5100
 Wire Wire Line
 	10200 5750 9700 5750
@@
 	2350 4500 4250 4500
 Wire Wire Line
-	1650 3100 2875 3100
-Wire Wire Line
-	2875 3100 2875 4800
-Wire Wire Line
-	2875 4800 4250 4800
-Wire Wire Line
-	1650 3000 2975 3000
-Wire Wire Line
-	2975 3000 2975 4700
-Wire Wire Line
-	2975 4700 4250 4700
+	1650 3100 2850 3100
+Wire Wire Line
+	2850 3100 2850 5200
+Wire Wire Line
+	1650 3000 2950 3000
+Wire Wire Line
+	2950 3000 2950 5100
 Wire Wire Line
 	1575 975  2300 975
@@
 	1700 1350 1575 1350
 Wire Wire Line
-	4175 4900 4250 4900
-Wire Wire Line
-	4250 5000 4150 5000
-Wire Wire Line
 	7600 4100 7450 4100
 Wire Wire Line
@@
 Wire Wire Line
 	3200 3400 4250 3400
+Wire Wire Line
+	9275 2800 10100 2800
+Wire Wire Line
+	7450 3300 9350 3300
+Wire Wire Line
+	9350 3300 9350 2900
+Wire Wire Line
+	9350 2900 10100 2900
+Wire Wire Line
+	2850 5200 4250 5200
+Wire Wire Line
+	2950 5100 4250 5100
+Wire Wire Line
+	2650 3300 2650 5000
+Wire Wire Line
+	2650 5000 4250 5000
+Wire Wire Line
+	2750 3200 2750 4900
+Wire Wire Line
+	2750 4900 4250 4900
+Wire Wire Line
+	4050 4700 4250 4700
+Wire Wire Line
+	4025 4800 4250 4800
 $EndSCHEMATC
