File: hardware/pcb/aero.kicad_pcb (KiCad board)
At the start: 4 copper layers, 89 parts, among them CON1 USB-MICRO-B, CON2 MMCX_CONN, J1 CORTEX_DBG_CONN, J2 LiPoly_Conn, Q1 Q_NPN_BEC, SW1 SW_PUSH, U1 STM32L151C8, U2 nRF8001, U3 ms5611, U4 BMX055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

Commit message: mega commit
Changed lines of the file:
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@@
   (segment (start 217.452 99.555) (end 217.437 99.555) (width 0.254) (layer F.Cu) (net 1))
   (segment (start 217.437 99.555) (end 216.166 100.826) (width 0.254) (layer F.Cu) (net 1))
-  (segment (start 210.07 98.425) (end 209.169 98.425) (width 0.2032) (layer F.Cu) (net 2) (status 400000))
-  (via (at 209.1055 98.4885) (size 0.635) (layers F.Cu B.Cu) (net 2))
-  (segment (start 209.169 98.425) (end 209.1055 98.4885) (width 0.2032) (layer F.Cu) (net 2))
+  (segment (start 210.07 98.425) (end 209.1182 98.425) (width 0.2032) (layer F.Cu) (net 2) (status 400000))
+  (via (at 209.042 98.5012) (size 0.635) (layers F.Cu B.Cu) (net 2))
+  (segment (start 209.1182 98.425) (end 209.042 98.5012) (width 0.2032) (layer F.Cu) (net 2))
   (segment (start 189.738 151.626) (end 189.726 151.626) (width 0.2032) (layer F.Cu) (net 2))
   (segment (start 189.726 151.626) (end 188.6585 150.5585) (width 0.2032) (layer F.Cu) (net 2))
@@
   (segment (start 227.9135 102.2985) (end 225.3735 102.2985) (width 0.254) (layer F.Cu) (net 14))
   (segment (start 225.3735 102.2985) (end 224.04 100.965) (width 0.254) (layer F.Cu) (net 14))
-  (segment (start 225.54 95.885) (end 227.85 95.885) (width 0.2032) (layer F.Cu) (net 16) (status C00000))
+  (segment (start 225.54 95.885) (end 227.85 95.885) (width 0.2032) (layer F.Cu) (net 16))
   (segment (start 184.642 156.21) (end 184.642 155.3812) (width 0.508) (layer F.Cu) (net 17))
   (segment (start 184.162 154.9012) (end 184.162 154.178) (width 0.508) (layer F.Cu) (net 17))

Commit message: Finished layout
Parts:
- added Ant_Bluetooth: VAL**, aero:Ant_Bluetooth, F.Cu at (191.8, 113.8)
- moved TP3 68.1 mm to (185.4, 147.8)
- moved AUD1 66.9 mm to (178.1, 143.4), turned to 225 degrees
- moved TP2 66.3 mm to (184.9, 142.2)
- moved R16 63.3 mm to (181.1, 144.4), turned to 270 degrees
- moved TP4 62.1 mm to (186.9, 142.2)
- moved Q1 52.3 mm to (183.4, 145.3), turned to 180 degrees
- moved TP1 50.1 mm to (162.6, 136.7)
- moved R15 50.1 mm to (182.3, 141.8)
- moved TP9 48.2 mm to (179.2, 125.7)
- moved TP10 47.8 mm to (180.9, 127.7)
- moved C11 47.2 mm to (174.1, 117.6)
- moved C12 47.2 mm to (174.1, 118.9)
- moved C13 47.2 mm to (170.3, 117.6)
- moved C14 47.2 mm to (170.3, 122.7)
- moved C16 47.2 mm to (174.8, 124.3)
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Connections:
- D3 pad 1: Net-(D3-Pad1) -> Net-(C33-Pad1)
- D3 pad 2: Net-(C33-Pad1) -> Net-(D3-Pad2)
- L4 pad 1: Net-(D3-Pad1) -> Net-(D3-Pad2)
- U5 pad : (no net) -> GND
- U6 pad 11: (no net) -> GND
- U8 pad 1: Net-(D3-Pad1) -> Net-(D3-Pad2)
Routing:
- net GND: track 69.1 -> 175.3 mm, vias 28 -> 89
- net Vbatt: track 7.43 -> 50.8 mm, vias 0 -> 2
- net /at45db321e/SCK: track 0.00 -> 34.9 mm, vias 0 -> 2
- net /bmx055/MISO: track 0.00 -> 33.9 mm, vias 0 -> 2
- net /at45db321e/MISO: track 0.00 -> 31.6 mm, vias 0 -> 3
- net ~NRST: track 2.79 -> 32.3 mm, vias 0 -> 2
- net /warn/PIEZO_EN: track 0.00 -> 29.1 mm, vias 0 -> 4
- net /bmx055/SCK: track 0.00 -> 28.6 mm, vias 0 -> 2
- net /bmx055/MOSI: track 0.00 -> 27.3 mm, vias 0 -> 2
- net /at45db321e/MOSI: track 0.00 -> 27.3 mm, vias 0 -> 3
- net /power/USB_D+: track 0.00 -> 25.6 mm, vias 0 -> 2
- net Net-(J1-Pad2): track 0.00 -> 25.2 mm, vias 0 -> 2
- net ~PG: track 0.00 -> 23.5 mm, vias 0 -> 2
- net +3V3: track 27.2 -> 49.4 mm, vias 10 -> 20
- net /ms5611/EN: track 2.20 -> 24.0 mm, vias 0 -> 3
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- added copper zone on F.Cu, net GND
- added copper zone on F.Cu, net Net-(C33-Pad1)
- added copper zone on F.Cu, net Net-(C33-Pad2)
- added copper zone on F.Cu, net Net-(D3-Pad2)
- added copper zone on F.Cu, net Vbatt
Other:
- board outline added: 39.1 x 46.2 mm
- board text added: "alti"
- board text added: "yan@srtd.org"

Commit message: fixed a few known pcb issues
Parts:
- moved C17 0.56 mm to (175.3, 114.9), turned to 270 degrees
- moved C18 0.14 mm to (180.3, 114.9), turned to 90 degrees
- moved Y4 0.11 mm to (177.9, 114.9), turned to 0 degrees
Connections:
- Y4 pad 2: Net-(C18-Pad2) -> GND
- Y4 pad 3: GND -> Net-(C18-Pad2)
Routing:
- net Net-(C18-Pad2): track 4.62 -> 7.46 mm
- net Net-(C17-Pad2): track 7.95 -> 5.63 mm
