File: hardware/pcb/aero.kicad_pcb (KiCad board)
At the start: 4 copper layers, 39.1 x 46.2 mm, 90 parts, among them CON1 USB-MICRO-B, CON2 MMCX_CONN, J1 CORTEX_DBG_CONN, J2 LiPoly_Conn, Q1 Q_NPN_BEC, SW1 SW_PUSH, U1 STM32L151C8, U2 nRF8001, U3 ms5611, U4 BMX055, U5 AT45DB321E, U6 BQ24040DSQ, U7 TPS783, U8 TPS61041, U9 ZXMHC6A07N8, Y1 Crystal, Y2 Crystal, Y3 32.768KHz, Y4 16MHz

Commit message: pre major restructuring commit
Parts:
- added REF**: TC2050-IDC-NL, aero:TC2050-IDC-NL, B.Cu at (197.5, 142.2)
Routing:
- net GND: track 174.8 -> 288.5 mm, vias 89 -> 86
- net /at45db321e/MISO: track 31.6 -> 7.79 mm, vias 3 -> 1
- net ~PG: track 23.5 -> 0.95 mm, vias 2 -> 0
- net ACC_INT: track 19.7 -> 1.59 mm, vias 2 -> 0
- net /power/USB_D-: track 20.0 -> 4.33 mm, vias 2 -> 1
- net Net-(R2-Pad1): track 15.1 -> 1.30 mm, vias 2 -> 0
- net /warn/STATUS_LED: track 12.8 -> 2.04 mm, vias 2 -> 1
- net Net-(C10-Pad2): track 10.5 -> 2.91 mm, vias 2 -> 0

Commit message: more progress on new layout
Parts:
- removed Ant_Bluetooth: VAL**, aero:Ant_Bluetooth
- removed C32: 4.7uF, Capacitors_SMD:C_0603
- removed C33: 22pF, Capacitors_SMD:C_0603
- removed C34: 100nF, Capacitors_SMD:C_0603
- removed D3: D_Schottky, Diodes_SMD:SOD-123
- removed L3: 5.6nH, Capacitors_SMD:C_0603
- removed L4: 10u, aero:SDR0703
- removed R15: 3k, Resistors_SMD:R_0603
- removed R16: 2k, Resistors_SMD:R_0603
- removed REF**: TC2050-IDC-NL, aero:TC2050-IDC-NL
- removed TP10, TP7, TP8, TP9: Test_Point, aero:TP_0603
- removed Y4: 16MHz, aero:crystal_SMD_3225
- added A1: 2450AT18A100, aero:2450AT18A100, F.Cu at (112.3, 17.8)
- added A2: U.FL_Antenna, aero:U.FL, F.Cu at (137.0, 18.9)
- added U10: BU4SU69G2, aero:SSOP-5, F.Cu at (111.8, 77.5)
- added U11: BU4SU69G2, aero:SSOP-5, F.Cu at (113.0, 80.6)
- added U12: NC7WZ17, Housings_SOT-23_SOT-143_TSOT-6:SC-70-6, F.Cu at (110.1, 123.5)
- added U13: u-blox_max-7c/q, aero:ublox_MAX7, F.Cu at (132.3, 28.6)
- added U14: MAX2659, aero:6-µDFN, F.Cu at (132.7, 20.8)
- C1, C2, C3, C4, C5, C6, C7, C8: footprint Capacitors_SMD:C_0603 -> Capacitors_SMD:C_0402
- C10, C14, C9: value 15pF -> 100nF; footprint Capacitors_SMD:C_0603 -> Capacitors_SMD:C_0402
- C11, C12: value 100nF -> 15pF; footprint Capacitors_SMD:C_0603 -> Capacitors_SMD:C_0402
- C13: value 15pF -> 33nF; footprint Capacitors_SMD:C_0603 -> Capacitors_SMD:C_0402
- C15: value 33nF -> 12pF; footprint Capacitors_SMD:C_0603 -> Capacitors_SMD:C_0402
- C16: value 100nF -> 12pF; footprint Capacitors_SMD:C_0603 -> Capacitors_SMD:C_0402
- C17: value 12pF -> 1.0nF; footprint Capacitors_SMD:C_0603 -> Capacitors_SMD:C_0402
- C18: value 12pF -> 2.2nF; footprint Capacitors_SMD:C_0603 -> Capacitors_SMD:C_0402
- C19: value 1.0nF -> 100nF; footprint Capacitors_SMD:C_0603 -> Capacitors_SMD:C_0402
- C20: value 2.2nF -> 100nF; footprint Capacitors_SMD:C_0603 -> Capacitors_SMD:C_0402
- C21: value NC -> 100nF; footprint Capacitors_SMD:C_0603 -> Capacitors_SMD:C_0402
- C22: value 1.8pF -> 100nF; footprint Capacitors_SMD:C_0603 -> Capacitors_SMD:C_0402
- C23: value 1.2pF -> 1uF; footprint Capacitors_SMD:C_0603 -> Capacitors_SMD:C_0402
- C24, C25: value 100nF -> 1uF; footprint Capacitors_SMD:C_0603 -> Capacitors_SMD:C_0402
- C26: value 100nF -> 2.2uF; footprint Capacitors_SMD:C_0603 -> Capacitors_SMD:C_0402
- C27: value 100nF -> 4.7uF; footprint Capacitors_SMD:C_0603 -> Capacitors_SMD:C_0402
- C28: value 1uF -> 22pF; footprint Capacitors_SMD:C_0603 -> Capacitors_SMD:C_0402
- C29: value 1uF -> 100nF; footprint Capacitors_SMD:C_0603 -> Capacitors_SMD:C_0402
- C30: value 1uF -> 33nF; footprint Capacitors_SMD:C_0603 -> Capacitors_SMD:C_0402
- C31: value 2.2uF -> 470pF; footprint Capacitors_SMD:C_0603 -> Capacitors_SMD:C_0402
- D2: value LED -> D_Schottky; footprint LEDs:LED-0805 -> Diodes_SMD:SOD-123
- J1: footprint aero:FTSH-105-01 -> aero:TC2050-IDC-NL; moved to B.Cu
- J2: footprint Capacitors_SMD:C_1206_HandSoldering -> aero:Conn_Molex_78171-02; moved to B.Cu
- JP1, JP2: footprint aero:Pin_Header_1x02 -> aero:Pin_Header_1x02_2mm
- L1: value 8.2nH -> 10u; footprint Capacitors_SMD:C_0603 -> aero:IND-744029100
- L2: value 3.9nH -> 6.8nH; footprint Capacitors_SMD:C_0603 -> Capacitors_SMD:C_0402
- Q1: value Q_NPN_BEC -> BSS138
- R1, R2: footprint Resistors_SMD:R_0603 -> Resistors_SMD:R_0402
- R10: value 22 -> 200; footprint Resistors_SMD:R_0603 -> Resistors_SMD:R_0402
- R11: value 10k -> 2.21m; footprint Resistors_SMD:R_0603 -> Resistors_SMD:R_0402
- R12: value 120 -> 309k; footprint Resistors_SMD:R_0603 -> Resistors_SMD:R_0402
- R13: value 2.21m -> 30k; footprint Resistors_SMD:R_0603 -> Resistors_SMD:R_0402
- R14: value 140k -> 10k; footprint Resistors_SMD:R_0603 -> Resistors_SMD:R_0402
- R3: value 220 -> 1.5k; footprint Resistors_SMD:R_0603 -> Resistors_SMD:R_0402
- R4: value 1.5k -> 22k; footprint Resistors_SMD:R_0603 -> Resistors_SMD:R_0402
- R5: value 1.5k -> 825; footprint Resistors_SMD:R_0603 -> Resistors_SMD:R_0402
- R6: value 22k -> 2k; footprint Resistors_SMD:R_0603 -> Resistors_SMD:R_0402
- R7: value 825 -> 22; footprint Resistors_SMD:R_0603 -> Resistors_SMD:R_0402
- R8: value 2k -> 22; footprint Resistors_SMD:R_0603 -> Resistors_SMD:R_0402
- R9: value 22 -> 10k; footprint Resistors_SMD:R_0603 -> Resistors_SMD:R_0402
- U2: footprint Housings_DFN_QFN:QFN-32-1EP_5x5mm_Pitch0.5mm -> aero:QFN-32-1EP_5x5mm_Pitch0.5mm
- U3: value ms5611 -> 2450BM14A0002; footprint aero:ms5611 -> aero:2450BM14A0002
- U4: value BMX055 -> ms5611; footprint aero:BMX055 -> aero:ms5611
- U5: value AT45DB321E -> BMX055; footprint aero:UDFN-8 -> aero:BMX055
- U6: value BQ24040DSQ -> AT45DB321E; footprint aero:WSON-10-1EP -> aero:UDFN-8
- U7: value TPS783 -> BQ24040DSQ; footprint Housings_SOT-23_SOT-143_TSOT-6:SOT-23-5 -> aero:WSON-10-1EP
- U8: value TPS61041 -> TPS783
- U9: value ZXMHC6A07N8 -> TPS61041; footprint Power_Integrations:SO-8 -> Housings_SOT-23_SOT-143_TSOT-6:SOT-23-5
- Y1: footprint aero:FC-135R -> aero:Crystal_32768_FC-135R
- Y2: value Crystal -> 32.768KHz; footprint aero:Murata_CSTCE-G_Oscillator -> aero:Crystal_32768_FC-135R
- Y3: value 32.768KHz -> 16MHz; footprint aero:FC-135R -> aero:Crystal_TSX_3225
- moved C31 145.3 mm to (132.7, 19.3), turned to 0 degrees
- moved R4 144.6 mm to (112.8, 20.3), turned to 270 degrees
- moved C30 142.6 mm to (130.5, 21.1), turned to 180 degrees
- moved C9 137.6 mm to (111.2, 20.4), turned to 90 degrees
- moved R14 129.5 mm to (130.6, 22.2), turned to 180 degrees
- moved C10 125.3 mm to (114.4, 25.9), turned to 270 degrees
- moved Y2 123.9 mm to (116.8, 27.9), turned to 0 degrees
- moved U3 117.6 mm to (115.6, 17.9), turned to 90 degrees
- moved U2 117.3 mm to (116.1, 22.1), turned to 90 degrees
- moved C18 115.7 mm to (117.4, 17.8), turned to 0 degrees
- moved C14 114.9 mm to (113.1, 23.0), turned to 270 degrees
- moved C15 114.5 mm to (111.6, 24.1)
- moved C16 114.5 mm to (112.0, 28.6), turned to 0 degrees
- moved L2 114.1 mm to (133.1, 18.2)
- moved C17 113.7 mm to (112.0, 20.4), turned to 90 degrees
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Connections:
- C1 pad 1: +3V3 -> +3V
- C10 pad 1: GND -> Net-(C10-Pad1)
- C10 pad 2: Net-(C10-Pad2) -> GND
- C11 pad 1: +3V3 -> Net-(C11-Pad1)
- C14 pad 1: Net-(C14-Pad1) -> +3V
- C15 pad 1: Net-(C15-Pad1) -> GND
- C15 pad 2: GND -> Net-(C15-Pad2)
- C16 pad 1: +3V3 -> GND
- C16 pad 2: GND -> Net-(C16-Pad2)
- C17 pad 1: GND -> +3V
- C17 pad 2: Net-(C17-Pad2) -> GND
- C18 pad 1: GND -> Net-(C18-Pad1)
- C18 pad 2: Net-(C18-Pad2) -> GND
- C19 pad 1: +3V3 -> +3V
- C2 pad 1: +3V3 -> +3V
- C20 pad 1: Net-(C20-Pad1) -> +3V
- C21 pad 1: Net-(C20-Pad1) -> +3V
- C22 pad 1: /nRF8001/Antenna -> +3V
- C22 pad 2: Net-(C22-Pad2) -> GND
- C23 pad 1: /nRF8001/Antenna -> Net-(C23-Pad1)
- C24 pad 1: +3V3 -> Net-(C24-Pad1)
- C25 pad 1: +3V3 -> Vbatt
- C26 pad 1: +3V3 -> +3V
- C27 pad 1: +3V3 -> Vbatt
- C28 pad 1: Net-(C28-Pad1) -> +10V
- C28 pad 2: GND -> Net-(C28-Pad2)
- C29 pad 1: Net-(C29-Pad1) -> +10V
- C3 pad 1: +3V3 -> +3V
- C30 pad 1: Vbatt -> Net-(C30-Pad1)
- C31 pad 1: +3V3 -> Net-(C31-Pad1)
- C31 pad 2: GND -> Net-(C31-Pad2)
- C4 pad 1: +3V3 -> +3V
- C5 pad 1: +3V3 -> +3V
- C9 pad 1: Net-(C9-Pad1) -> +3V
- CON1 pad 1: Net-(C29-Pad1) -> Net-(C24-Pad1)
- CON2 pad 1: Net-(CON2-Pad2) -> Net-(CON2-Pad1)
- CON2 pad 2: Net-(CON2-Pad1) -> Net-(CON2-Pad2)
- D1 pad 2: /power/~CHG -> /warn/STATUS_LED
- D2 pad 1: /warn/STATUS_LED -> +10V
- J1 pad 1: +3V3 -> +3V
- JP1 pad 1: Net-(C29-Pad1) -> Net-(C24-Pad1)
- JP1 pad 2: Net-(C28-Pad1) -> Net-(C23-Pad1)
- L1 pad 1: Net-(L1-Pad1) -> Net-(D2-Pad2)
- L1 pad 2: Net-(L1-Pad2) -> Vbatt
- L2 pad 1: Net-(L1-Pad2) -> Net-(C31-Pad2)
- L2 pad 2: Net-(C22-Pad2) -> Net-(A2-Pad1)
- Q1 pad 1: Net-(Q1-Pad1) -> /warn/PIEZO_OUT
- Q1 pad 3: Net-(AUD1-Pad2) -> Net-(Q1-Pad3)
- R10 pad 1: /power/USB_D+ -> GND
- R10 pad 2: Net-(CON1-Pad3) -> Net-(D1-Pad1)
- R11 pad 1: GND -> +10V
- R11 pad 2: Net-(R11-Pad2) -> Net-(C28-Pad2)
- R12 pad 1: GND -> Net-(C28-Pad2)
- R12 pad 2: Net-(D2-Pad2) -> GND
- R13 pad 1: Net-(C33-Pad1) -> +10V
- R13 pad 2: Net-(C33-Pad2) -> Net-(Q1-Pad3)
- R14 pad 1: Net-(C33-Pad2) -> Net-(R14-Pad1)
- R3 pad 1: Net-(C9-Pad1) -> +3V
- R3 pad 2: Net-(R3-Pad2) -> /power/USB_D+
- R4 pad 1: +3V3 -> GND
- R4 pad 2: /power/USB_D+ -> Net-(R4-Pad2)
- R5 pad 1: GND -> Net-(R5-Pad1)
- R5 pad 2: Net-(D1-Pad1) -> GND
- R6 pad 1: GND -> Net-(R6-Pad1)
- R6 pad 2: Net-(R6-Pad2) -> GND
- R7 pad 1: Net-(R7-Pad1) -> /power/USB_D-
- R7 pad 2: GND -> Net-(CON1-Pad2)
- R8 pad 1: Net-(R8-Pad1) -> /power/USB_D+
- R8 pad 2: GND -> Net-(CON1-Pad3)
- R9 pad 1: /power/USB_D- -> GND
- R9 pad 2: Net-(CON1-Pad2) -> Net-(R9-Pad2)
- TP1 pad 1: /warn/PIEZO_EN -> /bmx055/SCK
- TP2 pad 1: /warn/PIEZO_OUT -> /bmx055/MISO
- TP3 pad 1: /warn/WARN_LED_A -> /bmx055/MOSI
- TP4 pad 1: /warn/WARN_LED_B -> /at45db321e/SCK
- TP5 pad 1: /bmx055/SCK -> /at45db321e/MOSI
- TP6 pad 1: /bmx055/MISO -> /at45db321e/MISO
- U1 pad 1: +3V3 -> +3V
- U1 pad 18: Net-(U1-Pad18) -> /bmx055/ACC_SEL
- U1 pad 19: ~PG -> /bmx055/GYRO_SEL
- U1 pad 2: Net-(U1-Pad2) -> /GPS/TIMEPULSE
- U1 pad 20: Net-(U1-Pad20) -> /bmx055/MAG_SEL
- U1 pad 24: +3V3 -> +3V
- U1 pad 29: MAG_SEL -> Net-(U1-Pad29)
- U1 pad 30: ACC_SEL -> ~PG
- U1 pad 31: GYRO_SEL -> ~CHG
- U1 pad 36: +3V3 -> +3V
- U1 pad 40: ACC_INT -> /warn/PIEZO_EN
- U1 pad 41: Net-(U1-Pad41) -> /warn/PIEZO_OUT
- U1 pad 42: /warn/PIEZO_EN -> /GPS/RxD
- U1 pad 43: /warn/PIEZO_OUT -> /GPS/TxD
- U1 pad 48: +3V3 -> +3V
- U1 pad 49: GND -> (no net)
- U1 pad 5: Net-(C10-Pad2) -> /GPS/RESET
- U1 pad 6: Net-(R3-Pad2) -> /GPS/EXT_INT
- U1 pad 9: +3V3 -> +3V
- U2 pad 1: +3V3 -> +3V
- U2 pad 2: Net-(C12-Pad1) -> Net-(C10-Pad1)
- U2 pad 20: Net-(C20-Pad1) -> Net-(C18-Pad1)
- U2 pad 21: Net-(L1-Pad1) -> Net-(U2-Pad21)
- U2 pad 22: Net-(L1-Pad2) -> Net-(U2-Pad22)
- U2 pad 24: +3V3 -> +3V
- U2 pad 25: Net-(R6-Pad2) -> Net-(R4-Pad2)
- U2 pad 26: +3V3 -> +3V
- U2 pad 27: Net-(C18-Pad2) -> Net-(C16-Pad2)
- U2 pad 28: Net-(C17-Pad2) -> Net-(C15-Pad2)
- U2 pad 29: +3V3 -> +3V
- U2 pad 3: Net-(C15-Pad1) -> Net-(C13-Pad1)
- U2 pad 4: Net-(C13-Pad1) -> Net-(C11-Pad1)
- U2 pad 5: Net-(C14-Pad1) -> Net-(C12-Pad1)
- U2 pad 9: +3V3 -> +3V
- U3 pad 1: +3V3 -> Net-(A1-Pad1)
- U3 pad 3: GND -> Net-(U2-Pad22)
- U3 pad 4: /ms5611/EN -> Net-(U2-Pad21)
- U3 pad 5: /ms5611/EN -> Net-(C18-Pad1)
- U3 pad 6: /bmx055/MISO -> Net-(U3-Pad6)
- U4 pad 1: Net-(U4-Pad1) -> +3V
- U4 pad 2: Net-(U4-Pad2) -> GND
- U4 pad 3: +3V3 -> GND
- U4 pad 4: GND -> /ms5611/EN
- U4 pad 5: GYRO_SEL -> /ms5611/EN
- U4 pad 6: GND -> /bmx055/MISO
- U4 pad 7: GND -> /bmx055/MOSI
- U4 pad 8: Net-(U4-Pad8) -> /bmx055/SCK
- U5 pad 1: /at45db321e/MOSI -> Net-(U5-Pad1)
- U5 pad 2: /at45db321e/SCK -> Net-(U5-Pad2)
- U5 pad 3: /at45db321e/~RESET -> +3V
- U5 pad 4: /at45db321e/~CS -> GND
- U5 pad 5: +3V3 -> /bmx055/GYRO_SEL
- U5 pad 6: +3V3 -> GND
- U5 pad 8: /at45db321e/MISO -> Net-(U5-Pad8)
- U6 pad 1: Net-(C28-Pad1) -> /at45db321e/MOSI
- U6 pad 2: Net-(R7-Pad1) -> /at45db321e/SCK
- U6 pad 3: GND -> /at45db321e/~RESET
- U6 pad 4: Net-(R8-Pad1) -> /at45db321e/~CS
- U6 pad 5: ~PG -> +3V
- U6 pad 6: Net-(U6-Pad6) -> +3V
- U6 pad 7: Net-(U6-Pad7) -> GND
- U6 pad 8: /power/~CHG -> /at45db321e/MISO
- U7 pad 1: Vbatt -> Net-(C23-Pad1)
- U7 pad 2: GND -> Net-(R5-Pad1)
- U7 pad 3: Vbatt -> GND
- U7 pad 4: GND -> Net-(R6-Pad1)
- U7 pad 5: +3V3 -> ~PG
- U8 pad 1: Net-(D3-Pad2) -> Vbatt
- U8 pad 3: Net-(C33-Pad2) -> Vbatt
- U8 pad 4: /warn/PIEZO_EN -> GND
- U8 pad 5: Vbatt -> +3V
- U9 pad 1: /warn/WARN_LED_B -> Net-(D2-Pad2)
- U9 pad 2: Net-(CON2-Pad1) -> GND
- U9 pad 3: GND -> Net-(C28-Pad2)
- U9 pad 4: /warn/WARN_LED_A -> /warn/PIEZO_EN
- U9 pad 5: /warn/WARN_LED_A -> Vbatt
- Y2 pad 1: Net-(C9-Pad1) -> Net-(C11-Pad1)
- Y2 pad 2: Net-(C10-Pad2) -> Net-(C12-Pad1)
- Y3 pad 1: Net-(C13-Pad1) -> Net-(C15-Pad2)
- Y3 pad 2: Net-(C14-Pad1) -> Net-(C16-Pad2)
Routing:
- net GND: track 288.5 -> 0.00 mm, vias 86 -> 0
- net Vbatt: track 50.8 -> 0.00 mm, vias 2 -> 0
- net +3V3: track 49.4 -> 0.00 mm, vias 20 -> 0
- net /at45db321e/SCK: track 34.9 -> 0.00 mm, vias 2 -> 0
- net /bmx055/MISO: track 33.9 -> 0.00 mm, vias 2 -> 0
- net ~NRST: track 32.3 -> 0.00 mm, vias 2 -> 0
- net /warn/PIEZO_EN: track 29.1 -> 0.00 mm, vias 4 -> 0
- net /bmx055/SCK: track 28.6 -> 0.00 mm, vias 2 -> 0
- net /bmx055/MOSI: track 27.3 -> 0.00 mm, vias 2 -> 0
- net /at45db321e/MOSI: track 27.3 -> 0.00 mm, vias 3 -> 0
- net /power/USB_D+: track 25.6 -> 0.00 mm, vias 2 -> 0
- net Net-(J1-Pad2): track 25.2 -> 0.00 mm, vias 2 -> 0
- net /ms5611/EN: track 24.0 -> 0.00 mm, vias 3 -> 0
- net Net-(CON2-Pad2): track 21.5 -> 0.00 mm
- net GYRO_SEL: track 21.3 -> 0.00 mm
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- removed copper zone on In2.Cu, net +3V3
- removed copper zone on F.Cu, net GND
- removed copper zone on In1.Cu, net GND
- removed copper zone on F.Cu, net Net-(C33-Pad1)
- removed copper zone on F.Cu, net Net-(C33-Pad2)
- removed copper zone on F.Cu, net Net-(D3-Pad2)
- removed copper zone on F.Cu, net Vbatt
Other:
- board outline removed
- net class Default: clearance 0.1524 -> 0.2; trace_width 0.1524 -> 0.25; via_dia 0.635 -> 0.6; via_drill 0.381 -> 0.4
- rule trace_clearance: 0.1524 -> 0.2
- rule via_min_drill: 0.381 -> 0.254
- rule via_min_size: 0.635 -> 0.3556
- board text removed: "alti"
- board text removed: "yan@srtd.org"

Commit message: more pcb rework
Parts:
- added REF**: v, aero:Via_Stitch, F.Cu at (186.4, 38.6)
- moved J1 90.2 mm to (131.2, 97.3), turned to 270 degrees
- moved U12 89.1 mm to (198.2, 136.9), turned to 180 degrees
- moved CON2 89.1 mm to (194.0, 138.0)
- moved A1 87.8 mm to (198.1, 36.6), turned to 90 degrees
- moved C9 86.0 mm to (195.2, 39.2), turned to 0 degrees
- moved U3 86.0 mm to (197.7, 43.6), turned to 0 degrees
- moved C17 85.5 mm to (195.2, 39.9), turned to 0 degrees
- moved C18 85.0 mm to (197.8, 45.4), turned to 270 degrees
- moved R4 85.0 mm to (195.3, 40.8), turned to 180 degrees
- moved C14 81.6 mm to (192.6, 41.1), turned to 180 degrees
- moved C22 81.5 mm to (198.6, 52.0)
- moved C15 81.3 mm to (191.5, 39.6), turned to 90 degrees
- moved U6 80.7 mm to (193.8, 52.7)
- moved U2 80.4 mm to (193.5, 44.1), turned to 0 degrees
- moved Y3 78.3 mm to (189.2, 40.0), turned to 180 degrees
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Routing:
- net +10V: track 2.94 -> 0.00 mm
- net Net-(C12-Pad1): track 1.42 -> 0.00 mm
- net (no net): track 1.42 -> 0.00 mm
- net Net-(C23-Pad1): track 0.89 -> 0.00 mm
- net Net-(R14-Pad1): track 0.68 -> 0.00 mm
Other:
- board text added: "08.2015"
- board text added: "Alti v0.2"
- board text added: "yan@srtd.org"

Commit message: ver2 is nearing completion.
Parts:
- removed REF**: v, aero:Via_Stitch
- added C32: 100nF, Capacitors_SMD:C_0402, F.Cu at (143.1, 91.8)
- added R15: 10m, Resistors_SMD:R_0402, F.Cu at (140.5, 91.8)
- added R16: 10m, Resistors_SMD:R_0402, F.Cu at (141.9, 91.8)
- added REF**11101: v, aero:Via_Stitch, F.Cu at (141.4, 74.6)
- added REF**11102: v, aero:Via_Stitch, F.Cu at (141.4, 75.6)
- added REF**11103: v, aero:Via_Stitch, F.Cu at (141.4, 76.6)
- added REF**11104: v, aero:Via_Stitch, F.Cu at (141.4, 77.6)
- added REF**11105: v, aero:Via_Stitch, F.Cu at (141.4, 78.6)
- added REF**11106: v, aero:Via_Stitch, F.Cu at (141.5, 79.6)
- added REF**1111: v, aero:Via_Stitch, F.Cu at (134.3, 74.6)
- added REF**11110: v, aero:Via_Stitch, F.Cu at (134.3, 83.6)
- added REF**111101: v, aero:Via_Stitch, F.Cu at (135.5, 113.8)
- added REF**11111: v, aero:Via_Stitch, F.Cu at (126.5, 113.8)
- added REF**11111111: v, aero:Via_Stitch, F.Cu at (128.0, 80.4)
- added REF**11111111: v, aero:Via_Stitch, F.Cu at (128.0, 79.7)
- added REF**11111111: v, aero:Via_Stitch, F.Cu at (128.0, 79.0)
- added REF**11111112: v, aero:Via_Stitch, F.Cu at (129.3, 80.6)
- added REF**11111112: v, aero:Via_Stitch, F.Cu at (129.3, 79.9)
- added REF**11111112: v, aero:Via_Stitch, F.Cu at (129.3, 79.2)
- added REF**11111112: v, aero:Via_Stitch, F.Cu at (128.0, 78.3)
- added REF**11111113: v, aero:Via_Stitch, F.Cu at (128.7, 80.6)
- added REF**11111113: v, aero:Via_Stitch, F.Cu at (128.7, 79.9)
- added REF**11111113: v, aero:Via_Stitch, F.Cu at (128.7, 79.2)
- added REF**11111113: v, aero:Via_Stitch, F.Cu at (129.7, 77.7)
- added REF**11111113: v, aero:Via_Stitch, F.Cu at (128.0, 77.7)
- added REF**11111114: v, aero:Via_Stitch, F.Cu at (129.7, 77.0)
- added REF**11111114: v, aero:Via_Stitch, F.Cu at (128.0, 77.0)
- added REF**11111115: v, aero:Via_Stitch, F.Cu at (130.4, 76.4)
- added REF**11111115: v, aero:Via_Stitch, F.Cu at (129.7, 76.4)
- added REF**11111115: v, aero:Via_Stitch, F.Cu at (128.0, 76.4)
- added REF**11111116: v, aero:Via_Stitch, F.Cu at (130.4, 75.8)
- added REF**11111116: v, aero:Via_Stitch, F.Cu at (129.7, 75.7)
- added REF**11111116: v, aero:Via_Stitch, F.Cu at (128.0, 75.7)
- added REF**11111117: v, aero:Via_Stitch, F.Cu at (130.4, 75.1)
- added REF**11111117: v, aero:Via_Stitch, F.Cu at (129.7, 75.1)
- added REF**11111117: v, aero:Via_Stitch, F.Cu at (128.0, 75.1)
- added REF**11111118: v, aero:Via_Stitch, F.Cu at (130.4, 74.5)
- added REF**11111118: v, aero:Via_Stitch, F.Cu at (129.7, 74.4)
- added REF**11111118: v, aero:Via_Stitch, F.Cu at (128.0, 74.4)
- added REF**1112: v, aero:Via_Stitch, F.Cu at (134.3, 75.6)
- added REF**11121: v, aero:Via_Stitch, F.Cu at (127.5, 113.8)
- added REF**1113: v, aero:Via_Stitch, F.Cu at (134.3, 76.6)
- added REF**11131: v, aero:Via_Stitch, F.Cu at (128.5, 113.8)
- added REF**11141: v, aero:Via_Stitch, F.Cu at (129.5, 113.8)
- added REF**11151: v, aero:Via_Stitch, F.Cu at (130.5, 113.8)
- added REF**1116: v, aero:Via_Stitch, F.Cu at (134.3, 79.6)
- added REF**11161: v, aero:Via_Stitch, F.Cu at (131.5, 113.8)
- added REF**1117: v, aero:Via_Stitch, F.Cu at (134.3, 80.6)
- added REF**11171: v, aero:Via_Stitch, F.Cu at (132.5, 113.8)
- added REF**1118: v, aero:Via_Stitch, F.Cu at (134.3, 81.6)
- added REF**11181: v, aero:Via_Stitch, F.Cu at (133.5, 113.8)
- added REF**1119: v, aero:Via_Stitch, F.Cu at (134.3, 82.6)
- added REF**11191: v, aero:Via_Stitch, F.Cu at (134.5, 113.8)
- added REF**1121: v, aero:Via_Stitch, F.Cu at (135.1, 74.6)
- added REF**11210: v, aero:Via_Stitch, F.Cu at (135.1, 83.6)
- added REF**1122: v, aero:Via_Stitch, F.Cu at (135.1, 75.6)
- added REF**1123: v, aero:Via_Stitch, F.Cu at (135.1, 76.6)
- added REF**1124: v, aero:Via_Stitch, F.Cu at (135.1, 77.6)
- added REF**1126: v, aero:Via_Stitch, F.Cu at (135.1, 79.9)
- added REF**1127: v, aero:Via_Stitch, F.Cu at (135.1, 80.6)
- added REF**1128: v, aero:Via_Stitch, F.Cu at (135.1, 81.6)
- added REF**1129: v, aero:Via_Stitch, F.Cu at (135.1, 82.6)
- added REF**1131: v, aero:Via_Stitch, F.Cu at (135.9, 74.6)
- added REF**11310: v, aero:Via_Stitch, F.Cu at (135.7, 83.6)
- added REF**1132: v, aero:Via_Stitch, F.Cu at (135.9, 75.6)
- added REF**1133: v, aero:Via_Stitch, F.Cu at (135.9, 76.6)
- added REF**1134: v, aero:Via_Stitch, F.Cu at (135.9, 77.6)
- added REF**1135: v, aero:Via_Stitch, F.Cu at (135.9, 78.6)
- added REF**1138: v, aero:Via_Stitch, F.Cu at (135.7, 81.6)
- added REF**1139: v, aero:Via_Stitch, F.Cu at (135.7, 82.6)
- added REF**1141: v, aero:Via_Stitch, F.Cu at (136.7, 74.6)
- added REF**11410: v, aero:Via_Stitch, F.Cu at (136.7, 83.6)
- added REF**1142: v, aero:Via_Stitch, F.Cu at (136.7, 75.6)
- added REF**1143: v, aero:Via_Stitch, F.Cu at (136.7, 76.6)
- added REF**1144: v, aero:Via_Stitch, F.Cu at (136.7, 77.6)
- added REF**1145: v, aero:Via_Stitch, F.Cu at (136.7, 78.6)
- added REF**1146: v, aero:Via_Stitch, F.Cu at (136.7, 79.6)
- added REF**1147: v, aero:Via_Stitch, F.Cu at (136.7, 80.6)
- added REF**1148: v, aero:Via_Stitch, F.Cu at (136.7, 81.6)
- added REF**1149: v, aero:Via_Stitch, F.Cu at (136.7, 82.6)
- added REF**1151: v, aero:Via_Stitch, F.Cu at (137.5, 74.6)
- added REF**11510: v, aero:Via_Stitch, F.Cu at (137.5, 83.6)
- added REF**1152: v, aero:Via_Stitch, F.Cu at (137.5, 75.6)
- added REF**1153: v, aero:Via_Stitch, F.Cu at (137.5, 76.6)
- added REF**1154: v, aero:Via_Stitch, F.Cu at (137.5, 77.6)
- added REF**1155: v, aero:Via_Stitch, F.Cu at (137.5, 78.6)
- added REF**1156: v, aero:Via_Stitch, F.Cu at (137.5, 79.6)
- added REF**1157: v, aero:Via_Stitch, F.Cu at (137.5, 80.6)
- added REF**1158: v, aero:Via_Stitch, F.Cu at (137.5, 81.6)
- added REF**1159: v, aero:Via_Stitch, F.Cu at (137.5, 82.6)
- added REF**1161: v, aero:Via_Stitch, F.Cu at (138.3, 74.6)
- added REF**11610: v, aero:Via_Stitch, F.Cu at (138.3, 83.6)
- added REF**11611: v, aero:Via_Stitch, F.Cu at (163.3, 80.3)
- added REF**11611: v, aero:Via_Stitch, F.Cu at (164.1, 80.2)
- added REF**11611: v, aero:Via_Stitch, F.Cu at (164.0, 77.6)
- added REF**11611: v, aero:Via_Stitch, F.Cu at (162.6, 77.6)
- added REF**11612: v, aero:Via_Stitch, F.Cu at (164.1, 79.6)
- added REF**11612: v, aero:Via_Stitch, F.Cu at (164.0, 77.0)
- added REF**11612: v, aero:Via_Stitch, F.Cu at (162.6, 77.0)
- added REF**11613: v, aero:Via_Stitch, F.Cu at (164.1, 78.9)
- added REF**11613: v, aero:Via_Stitch, F.Cu at (164.0, 76.3)
- added REF**11613: v, aero:Via_Stitch, F.Cu at (162.6, 76.3)
- added REF**11614: v, aero:Via_Stitch, F.Cu at (164.0, 75.7)
- added REF**11614: v, aero:Via_Stitch, F.Cu at (162.6, 75.7)
- added REF**11615: v, aero:Via_Stitch, F.Cu at (164.0, 75.0)
- added REF**11615: v, aero:Via_Stitch, F.Cu at (162.6, 75.0)
- added REF**11616: v, aero:Via_Stitch, F.Cu at (164.1, 80.9)
- added REF**11616: v, aero:Via_Stitch, F.Cu at (164.0, 78.2)
- added REF**11616: v, aero:Via_Stitch, F.Cu at (164.0, 74.4)
- added REF**11616: v, aero:Via_Stitch, F.Cu at (162.6, 74.4)
- added REF**1162: v, aero:Via_Stitch, F.Cu at (144.2, 76.6)
- added REF**1162: v, aero:Via_Stitch, F.Cu at (138.3, 75.6)
- added REF**1163: v, aero:Via_Stitch, F.Cu at (144.2, 77.6)
- added REF**1163: v, aero:Via_Stitch, F.Cu at (138.3, 76.6)
- added REF**1164: v, aero:Via_Stitch, F.Cu at (138.3, 77.6)
- added REF**1165: v, aero:Via_Stitch, F.Cu at (138.3, 78.6)
- added REF**1166: v, aero:Via_Stitch, F.Cu at (138.3, 79.6)
- added REF**1167: v, aero:Via_Stitch, F.Cu at (138.3, 80.6)
- added REF**1168: v, aero:Via_Stitch, F.Cu at (138.3, 81.6)
- added REF**1169: v, aero:Via_Stitch, F.Cu at (138.3, 82.6)
- added REF**1171: v, aero:Via_Stitch, F.Cu at (139.1, 74.6)
- added REF**11710: v, aero:Via_Stitch, F.Cu at (139.1, 83.6)
- added REF**11711: v, aero:Via_Stitch, F.Cu at (144.1, 79.6)
- added REF**117111: v, aero:Via_Stitch, F.Cu at (144.0, 80.9)
- added REF**117112: v, aero:Via_Stitch, F.Cu at (144.0, 81.5)
- added REF**117113: v, aero:Via_Stitch, F.Cu at (144.0, 82.2)
- added REF**117114: v, aero:Via_Stitch, F.Cu at (144.0, 82.8)
- added REF**1172: v, aero:Via_Stitch, F.Cu at (145.0, 76.6)
- added REF**1172: v, aero:Via_Stitch, F.Cu at (139.1, 75.6)
- added REF**11721: v, aero:Via_Stitch, F.Cu at (145.1, 79.6)
- added REF**117211: v, aero:Via_Stitch, F.Cu at (145.0, 80.9)
- added REF**117212: v, aero:Via_Stitch, F.Cu at (145.0, 81.5)
- added REF**117213: v, aero:Via_Stitch, F.Cu at (145.0, 82.2)
- added REF**117214: v, aero:Via_Stitch, F.Cu at (145.0, 82.8)
- added REF**1173: v, aero:Via_Stitch, F.Cu at (145.0, 77.6)
- added REF**1173: v, aero:Via_Stitch, F.Cu at (139.1, 76.6)
- added REF**11731: v, aero:Via_Stitch, F.Cu at (146.1, 79.6)
- added REF**117311: v, aero:Via_Stitch, F.Cu at (146.0, 80.9)
- added REF**117311111: v, aero:Via_Stitch, F.Cu at (151.0, 74.5)
- added REF**1173111110: v, aero:Via_Stitch, F.Cu at (151.0, 81.7)
- added REF**117311112: v, aero:Via_Stitch, F.Cu at (151.0, 75.3)
- added REF**117311113: v, aero:Via_Stitch, F.Cu at (151.0, 76.1)
- added REF**117311114: v, aero:Via_Stitch, F.Cu at (151.0, 76.9)
- added REF**117311115: v, aero:Via_Stitch, F.Cu at (151.0, 77.7)
- added REF**117311116: v, aero:Via_Stitch, F.Cu at (151.0, 78.5)
- added REF**117311117: v, aero:Via_Stitch, F.Cu at (151.0, 79.3)
- added REF**117311118: v, aero:Via_Stitch, F.Cu at (151.0, 80.1)
- added REF**117311119: v, aero:Via_Stitch, F.Cu at (151.0, 80.9)
- added REF**117312: v, aero:Via_Stitch, F.Cu at (146.0, 81.5)
- added REF**117313: v, aero:Via_Stitch, F.Cu at (146.0, 82.2)
- added REF**117314: v, aero:Via_Stitch, F.Cu at (146.0, 82.8)
- added REF**1174: v, aero:Via_Stitch, F.Cu at (145.0, 78.3)
- added REF**1174: v, aero:Via_Stitch, F.Cu at (139.1, 77.6)
- added REF**117411: v, aero:Via_Stitch, F.Cu at (147.0, 80.9)
- added REF**117412: v, aero:Via_Stitch, F.Cu at (147.0, 81.5)
- added REF**117413: v, aero:Via_Stitch, F.Cu at (147.0, 82.2)
- added REF**117414: v, aero:Via_Stitch, F.Cu at (147.0, 82.8)
- added REF**1175: v, aero:Via_Stitch, F.Cu at (139.1, 78.6)
- added REF**1176: v, aero:Via_Stitch, F.Cu at (139.1, 79.6)
- added REF**1177: v, aero:Via_Stitch, F.Cu at (139.1, 80.6)
- added REF**1178: v, aero:Via_Stitch, F.Cu at (139.1, 81.6)
- added REF**1179: v, aero:Via_Stitch, F.Cu at (139.1, 82.6)
- added REF**1181: v, aero:Via_Stitch, F.Cu at (139.9, 74.6)
- added REF**11810: v, aero:Via_Stitch, F.Cu at (139.9, 83.6)
- added REF**1182: v, aero:Via_Stitch, F.Cu at (139.9, 75.6)
- added REF**1183: v, aero:Via_Stitch, F.Cu at (145.8, 77.6)
- added REF**1183: v, aero:Via_Stitch, F.Cu at (139.9, 76.6)
- added REF**1184: v, aero:Via_Stitch, F.Cu at (145.8, 78.3)
- added REF**1184: v, aero:Via_Stitch, F.Cu at (139.9, 77.6)
- added REF**1185: v, aero:Via_Stitch, F.Cu at (139.9, 78.6)
- added REF**1186: v, aero:Via_Stitch, F.Cu at (139.9, 79.6)
- added REF**1187: v, aero:Via_Stitch, F.Cu at (139.9, 80.6)
- added REF**1188: v, aero:Via_Stitch, F.Cu at (139.9, 81.6)
- added REF**1189: v, aero:Via_Stitch, F.Cu at (139.9, 82.6)
- added REF**1191: v, aero:Via_Stitch, F.Cu at (140.7, 74.6)
- added REF**1192: v, aero:Via_Stitch, F.Cu at (140.7, 75.6)
- added REF**1193: v, aero:Via_Stitch, F.Cu at (140.7, 76.6)
- added REF**1194: v, aero:Via_Stitch, F.Cu at (140.7, 77.6)
- added REF**1195: v, aero:Via_Stitch, F.Cu at (140.7, 78.6)
- added REF**1196: v, aero:Via_Stitch, F.Cu at (140.7, 79.6)
- added REF**1197: v, aero:Via_Stitch, F.Cu at (140.7, 80.6)
- added REF**1198: v, aero:Via_Stitch, F.Cu at (140.7, 81.6)
- moved C7 70.3 mm to (155.1, 98.5), turned to 90 degrees
- moved Y1 65.9 mm to (156.8, 97.2), turned to 270 degrees
- moved R1 65.1 mm to (154.7, 95.5), turned to 180 degrees
- moved C6 64.2 mm to (157.4, 94.7), turned to 0 degrees
- moved TP1 63.6 mm to (133.8, 88.3), turned to 180 degrees
- moved TP2 62.4 mm to (135.5, 88.3), turned to 180 degrees
- moved TP3 61.1 mm to (137.3, 88.5), turned to 180 degrees
- moved U1 53.7 mm to (148.8, 94.2)
- moved C21 53.1 mm to (126.7, 83.5), turned to 90 degrees
- moved C3 51.7 mm to (145.4, 90.0)
- moved C13 50.5 mm to (154.0, 79.0), turned to 270 degrees
- moved C30 50.3 mm to (130.6, 79.4)
- moved U5 50.3 mm to (129.2, 84.5), turned to 180 degrees
- moved C31 50.3 mm to (128.8, 77.8)
- moved L2 50.3 mm to (128.8, 75.6)
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Connections:
- CON1 pad 10: (no net) -> GND
- CON1 pad 11: (no net) -> GND
- U1 pad 25: /ms5611/EN -> BATT_SENSE
- U1 pad 29: Net-(U1-Pad29) -> MS5611_EN
- U1 pad 30: ~PG -> GPS_RX
- U1 pad 31: ~CHG -> GPS_TX
- U1 pad 42: /GPS/RxD -> ~CHG
- U1 pad 43: /GPS/TxD -> ~PG
- U1 pad 49: (no net) -> GND
- U13 pad 2: /GPS/TxD -> GPS_TX
- U13 pad 3: /GPS/RxD -> GPS_RX
- U2 pad 33: (no net) -> GND
- U4 pad 4: /ms5611/EN -> MS5611_EN
- U4 pad 5: /ms5611/EN -> MS5611_EN
- U7 pad 11: (no net) -> GND
- Y3 pad 3: (no net) -> GND
- Y3 pad 4: (no net) -> GND
Routing:
- net GND: track 0.00 -> 80.7 mm, vias 0 -> 53
- net Vbatt: track 0.00 -> 54.5 mm, vias 0 -> 5
- net /at45db321e/MOSI: track 0.00 -> 46.5 mm, vias 0 -> 4
- net /at45db321e/SCK: track 0.00 -> 40.5 mm, vias 0 -> 2
- net /at45db321e/MISO: track 0.00 -> 38.1 mm, vias 0 -> 3
- net /bmx055/MOSI: track 0.00 -> 36.3 mm
- net ~NRST: track 0.00 -> 36.2 mm, vias 0 -> 2
- net /bmx055/MISO: track 0.00 -> 34.2 mm, vias 0 -> 3
- net /GPS/RESET: track 0.00 -> 29.5 mm, vias 0 -> 2
- net /GPS/TIMEPULSE: track 0.00 -> 29.2 mm, vias 0 -> 2
- net /bmx055/SCK: track 0.00 -> 28.4 mm, vias 0 -> 2
- net +3V: track 0.00 -> 25.9 mm, vias 0 -> 26
- net /nRF8001/~RESET: track 0.00 -> 25.6 mm, vias 0 -> 2
- net /GPS/EXT_INT: track 0.00 -> 25.5 mm, vias 0 -> 2
- net /bmx055/GYRO_SEL: track 0.00 -> 24.8 mm, vias 0 -> 2
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- added copper zone on In2.Cu, net +3V
- added copper zone on F.Cu, net GND
- added copper zone on In1.Cu, net GND
Other:
- board outline added: 41 x 50 mm
- net class Default: clearance 0.2 -> 0.1524
- rule trace_clearance: 0.2 -> 0.1524

Commit message: no more vias under pads
Parts:
- removed the REF**1162 at (144.2, 76.6)
- moved C10 2.34 mm to (152.4, 78.0)
- moved REF**1163 2.23 mm to (146.2, 76.6)
- moved REF**1172 0.38 mm to (145.4, 76.6)
- moved REF**1173 0.38 mm to (145.4, 77.6)
- moved REF**1174 0.38 mm to (145.4, 78.3)
- moved REF**1183 0.38 mm to (146.2, 77.6)
- moved REF**1184 0.38 mm to (146.2, 78.3)
- moved Y3 0.28 mm to (154.1, 75.7), turned to 90 degrees
Connections:
- U1 pad 2: /GPS/TIMEPULSE -> /GPS/RESET
- U1 pad 5: /GPS/RESET -> /GPS/TIMEPULSE
Routing:
- net GND: track 80.7 -> 118.1 mm, vias 53 -> 50
- net +3V: track 25.9 -> 40.7 mm, vias 26 -> 25
- net /GPS/TIMEPULSE: track 29.2 -> 25.2 mm
- net Net-(C16-Pad2): track 6.70 -> 9.68 mm
- net Net-(C15-Pad2): track 8.77 -> 5.94 mm
- net +10V: track 22.5 -> 20.1 mm, vias 0 -> 2
- net Net-(C10-Pad1): track 1.40 -> 3.43 mm
- net Net-(D2-Pad2): track 5.92 -> 5.40 mm, vias 2 -> 0
- net Net-(J1-Pad4): track 14.9 -> 15.4 mm

Commit message: pre-antenna reorg commit
Parts:
- removed the REF**11111112 at (129.3, 79.2)
- removed the REF**11111113 at (129.7, 77.7)
- removed the REF**11111113 at (128.0, 77.7)
- removed REF**11111114 (x2), REF**11111115 (x3), REF**11111116 (x3), REF**11111117 (x3), REF**11111118 (x3): v, aero:Via_Stitch
- added A3: U.FL_Antenna, aero:Chip_Antenna_W3011A, F.Cu at (126.7, 69.0)
- added R17: 0, Resistors_SMD:R_0402, F.Cu at (127.1, 72.2)
- added R18: 0, Resistors_SMD:R_0402, F.Cu at (127.5, 72.6)
- added REF**: MountingHole_3mm, Mounting_Holes:MountingHole_3mm, F.Cu at (148.3, 71.8)
- added REF**: MountingHole_3mm, Mounting_Holes:MountingHole_3mm, F.Cu at (148.3, 104.7)
- added REF**1111: v, aero:Via_Stitch, F.Cu at (128.5, 71.4)
- added REF**1111: v, aero:Via_Stitch, F.Cu at (132.3, 67.2)
- added REF**1111: v, aero:Via_Stitch, F.Cu at (132.3, 68.2)
- added REF**1111: v, aero:Via_Stitch, F.Cu at (132.3, 69.2)
- added REF**1111: v, aero:Via_Stitch, F.Cu at (130.5, 71.4)
- added REF**1111: v, aero:Via_Stitch, F.Cu at (131.5, 71.4)
- added REF**1111: v, aero:Via_Stitch, F.Cu at (129.5, 71.4)
- added REF**1111: v, aero:Via_Stitch, F.Cu at (132.3, 73.1)
- added REF**1111: v, aero:Via_Stitch, F.Cu at (131.3, 73.1)
- added REF**1111: v, aero:Via_Stitch, F.Cu at (130.5, 73.1)
- added REF**1111: v, aero:Via_Stitch, F.Cu at (129.5, 73.1)
- added REF**1111: v, aero:Via_Stitch, F.Cu at (128.5, 73.1)
- added REF**1111: v, aero:Via_Stitch, F.Cu at (132.3, 70.2)
- added REF**1111: v, aero:Via_Stitch, F.Cu at (136.7, 72.0)
- added REF**1111: v, aero:Via_Stitch, F.Cu at (136.7, 71.0)
- added REF**11111111: v, aero:Via_Stitch, F.Cu at (128.2, 73.7)
- added REF**11111111: v, aero:Via_Stitch, F.Cu at (128.6, 74.2)
- added REF**11111111: v, aero:Via_Stitch, F.Cu at (129.1, 74.8)
- added REF**11111111: v, aero:Via_Stitch, F.Cu at (127.2, 74.7)
- added REF**11111111: v, aero:Via_Stitch, F.Cu at (127.6, 75.2)
- added REF**11111111: v, aero:Via_Stitch, F.Cu at (128.1, 75.8)
- added REF**11111112: v, aero:Via_Stitch, F.Cu at (129.6, 75.2)
- added REF**11111112: v, aero:Via_Stitch, F.Cu at (128.6, 76.2)
- added REF**1121: v, aero:Via_Stitch, F.Cu at (127.5, 66.4)
- added REF**1131: v, aero:Via_Stitch, F.Cu at (128.3, 66.4)
- added REF**1141: v, aero:Via_Stitch, F.Cu at (129.1, 66.4)
- added REF**1151: v, aero:Via_Stitch, F.Cu at (133.2, 68.0)
- added REF**1151: v, aero:Via_Stitch, F.Cu at (129.9, 66.4)
- added REF**1161: v, aero:Via_Stitch, F.Cu at (134.0, 68.0)
- added REF**1161: v, aero:Via_Stitch, F.Cu at (130.7, 66.4)
- added REF**11611: v, aero:Via_Stitch, F.Cu at (156.8, 69.2)
- added REF**11612: v, aero:Via_Stitch, F.Cu at (156.8, 73.1)
- added REF**11612: v, aero:Via_Stitch, F.Cu at (156.8, 68.5)
- added REF**11613: v, aero:Via_Stitch, F.Cu at (156.8, 72.5)
- added REF**11613: v, aero:Via_Stitch, F.Cu at (156.8, 67.9)
- added REF**11614: v, aero:Via_Stitch, F.Cu at (156.8, 71.8)
- added REF**11614: v, aero:Via_Stitch, F.Cu at (156.8, 67.2)
- added REF**11615: v, aero:Via_Stitch, F.Cu at (156.8, 71.2)
- added REF**11615: v, aero:Via_Stitch, F.Cu at (156.8, 66.6)
- added REF**11616: v, aero:Via_Stitch, F.Cu at (156.8, 70.5)
- added REF**11616: v, aero:Via_Stitch, F.Cu at (156.8, 65.9)
- added REF**11616: v, aero:Via_Stitch, F.Cu at (156.8, 69.8)
- added REF**1163: v, aero:Via_Stitch, F.Cu at (146.2, 75.9)
- added REF**1171: v, aero:Via_Stitch, F.Cu at (134.8, 68.0)
- added REF**1171: v, aero:Via_Stitch, F.Cu at (131.5, 66.4)
- added REF**1172: v, aero:Via_Stitch, F.Cu at (145.4, 75.9)
- added REF**117311111: v, aero:Via_Stitch, F.Cu at (151.8, 73.5)
- added REF**117311111: v, aero:Via_Stitch, F.Cu at (151.6, 83.0)
- added REF**117311112: v, aero:Via_Stitch, F.Cu at (152.6, 73.5)
- added REF**117311112: v, aero:Via_Stitch, F.Cu at (152.4, 83.0)
- added REF**117311113: v, aero:Via_Stitch, F.Cu at (153.4, 73.5)
- added REF**117311113: v, aero:Via_Stitch, F.Cu at (153.2, 83.0)
- added REF**117311114: v, aero:Via_Stitch, F.Cu at (154.2, 73.5)
- added REF**1181: v, aero:Via_Stitch, F.Cu at (135.6, 68.0)
- added REF**1181: v, aero:Via_Stitch, F.Cu at (132.3, 66.4)
- added REF**1191: v, aero:Via_Stitch, F.Cu at (136.4, 68.0)
- moved A2 6.02 mm to (134.8, 71.4), turned to 270 degrees
- moved C31 2.43 mm to (128.8, 75.4), turned to 135 degrees
- moved L2 2.12 mm to (127.4, 74.0), turned to 135 degrees
- moved U14 1.55 mm to (130.6, 76.4), turned to 315 degrees
- moved C30 1.21 mm to (130.4, 78.2), turned to 135 degrees
Connections:
- A2 pad 2: (no net) -> GND
- L2 pad 2: Net-(A2-Pad1) -> Net-(L2-Pad2)
- U6 pad : (no net) -> GND
Routing:
- net GND: track 118.1 -> 129.2 mm, vias 50 -> 63
- net Net-(A2-Pad1): track 1.53 -> 5.88 mm
- net Net-(A3-Pad1): track 0.00 -> 1.32 mm
- net Net-(C30-Pad1): track 2.90 -> 4.06 mm
- net Net-(L2-Pad2): track 0.00 -> 1.09 mm
- net Net-(R14-Pad1): track 10.6 -> 11.5 mm
- net +3V: track 40.7 -> 41.6 mm
- net /GPS/EXT_INT: track 25.1 -> 24.5 mm
- net /bmx055/MISO: track 34.2 -> 34.8 mm
- net /GPS/TIMEPULSE: track 25.2 -> 24.6 mm
- net Net-(C31-Pad1): track 1.54 -> 1.00 mm
Other:
- outline, holes or cut-outs redrawn
