File: hardware/pcb/warn.sch (KiCad schematic (older format))
At the start: 14 parts

Commit message: schematic updates
Parts:
- removed D?: D_Schottky, symbol D_Schottky
- removed R?: R, symbol R
- added 1k, R?: R, symbol R
- added D?: LED, symbol LED
- gave numbers to parts that had none: 5
Connections:
- wire segments 31 -> 34
Other:
- note added: "Add a flyback diode?"
- note added: "EN needs to be at least\n1.2v"
- note added: "NOTE: Update R when LED is picked out"
Changed lines of the file:
@@
 Text HLabel 9400 2600 2    60   Input ~ 0
 WARN_LED_EN
-Text HLabel 9400 2800 2    60   Input ~ 0
+Text HLabel 1700 2800 0    60   Input ~ 0
 STATUS_LED
 $Comp
@@
 	1    7750 5650
 	1    0    0    -1
-$EndComp
-$Comp
-L D_Schottky D?
-U 1 1 55381395
-P 7450 5100
-F 0 "D?" H 7450 5200 50  0000 C CNN
-F 1 "D_Schottky" H 7450 5000 50  0000 C CNN
-F 2 "" H 7450 5100 60  0000 C CNN
-F 3 "" H 7450 5100 60  0000 C CNN
-	1    7450 5100
-	0    -1   -1   0
 $EndComp
 $Comp
@@
 $EndComp
 $Comp
-L INDUCTOR L?
+L INDUCTOR 10u
 U 1 1 553817A7
 P 2700 5450
-F 0 "L?" V 2650 5450 50  0000 C CNN
+F 0 "10u" V 2650 5450 50  0000 C CNN
 F 1 "INDUCTOR" V 2800 5450 50  0000 C CNN
 F 2 "" H 2700 5450 60  0000 C CNN
@@
 $EndComp
 $Comp
-L R R?
+L R 2.2m
 U 1 1 55381851
 P 4200 5750
-F 0 "R?" V 4280 5750 50  0000 C CNN
+F 0 "2.2m" V 4280 5750 50  0000 C CNN
 F 1 "R" V 4200 5750 50  0000 C CNN
 F 2 "" V 4130 5750 30  0000 C CNN
@@
 $EndComp
 $Comp
-L R R?
+L R 130k
 U 1 1 5538187A
 P 4200 6350
-F 0 "R?" V 4280 6350 50  0000 C CNN
+F 0 "130k" V 4280 6350 50  0000 C CNN
 F 1 "R" V 4200 6350 50  0000 C CNN
 F 2 "" V 4130 6350 30  0000 C CNN
@@
 $EndComp
 $Comp
-L C C?
+L C 22p
 U 1 1 553818B9
 P 4600 5750
-F 0 "C?" H 4625 5850 50  0000 L CNN
+F 0 "22p" H 4625 5850 50  0000 L CNN
 F 1 "C" H 4625 5650 50  0000 L CNN
 F 2 "" H 4638 5600 30  0000 C CNN
@@
 $EndComp
 $Comp
-L C C?
+L C 1u
 U 1 1 553818E7
 P 4950 5750
-F 0 "C?" H 4975 5850 50  0000 L CNN
+F 0 "1u" H 4975 5850 50  0000 L CNN
 F 1 "C" H 4975 5650 50  0000 L CNN
 F 2 "" H 4988 5600 30  0000 C CNN
 F 3 "" H 4950 5750 60  0000 C CNN
 	1    4950 5750
-	1    0    0    -1
-$EndComp
-$Comp
-L R R?
-U 1 1 55381929
-P 4950 6350
-F 0 "R?" V 5030 6350 50  0000 C CNN
-F 1 "R" V 4950 6350 50  0000 C CNN
-F 2 "" V 4880 6350 30  0000 C CNN
-F 3 "" H 4950 6350 30  0000 C CNN
-	1    4950 6350
 	1    0    0    -1
 $EndComp
@@
 	7850 5200 7850 5450
 Wire Wire Line
-	7850 5350 7450 5350
-Wire Wire Line
-	7450 5350 7450 5250
-Wire Wire Line
-	7450 4950 7450 4850
-Wire Wire Line
-	7450 4850 7850 4850
-Wire Wire Line
 	7850 4750 7850 5100
-Connection ~ 7850 5350
-Connection ~ 7850 4850
 Wire Wire Line
 	7450 5650 7550 5650
@@
 Connection ~ 4200 6100
 Wire Wire Line
-	1650 6700 4950 6700
+	4950 6700 1650 6700
 Wire Wire Line
 	3300 6700 3300 6550
@@
 Connection ~ 4600 5450
 Wire Wire Line
-	4950 6200 4950 5900
-Wire Wire Line
-	4950 6700 4950 6500
+	4950 5900 4950 6700
 Connection ~ 4200 6700
 Wire Wire Line
@@
 Wire Wire Line
 	7850 6050 7850 5850
+$Comp
+L LED D?
+U 1 1 55381AF7
+P 2150 2800
+F 0 "D?" H 2150 2900 50  0000 C CNN
+F 1 "LED" H 2150 2700 50  0000 C CNN
+F 2 "" H 2150 2800 60  0000 C CNN
+F 3 "" H 2150 2800 60  0000 C CNN
+	1    2150 2800
+	-1   0    0    1
+$EndComp
+$Comp
+L R R?
+U 1 1 55381B8F
+P 2850 2800
+F 0 "R?" V 2930 2800 50  0000 C CNN
+F 1 "R" V 2850 2800 50  0000 C CNN
+F 2 "" V 2780 2800 30  0000 C CNN
+F 3 "" H 2850 2800 30  0000 C CNN
+	1    2850 2800
+	0    1    1    0
+$EndComp
+$Comp
+L GND #PWR?
+U 1 1 55381C08
+P 3400 3000
+F 0 "#PWR?" H 3400 2750 50  0001 C CNN
+F 1 "GND" H 3400 2850 50  0000 C CNN
+F 2 "" H 3400 3000 60  0000 C CNN
+F 3 "" H 3400 3000 60  0000 C CNN
+	1    3400 3000
+	1    0    0    -1
+$EndComp
+Wire Wire Line
+	1700 2800 1950 2800
+Wire Wire Line
+	2350 2800 2700 2800
+Wire Wire Line
+	3000 2800 3400 2800
+Wire Wire Line
+	3400 2800 3400 3000
+$Comp
+L R 1k
+U 1 1 55387943
+P 7600 5150
+F 0 "1k" V 7680 5150 50  0000 C CNN
+F 1 "R" V 7600 5150 50  0000 C CNN
+F 2 "" V 7530 5150 30  0000 C CNN
+F 3 "" H 7600 5150 30  0000 C CNN
+	1    7600 5150
+	1    0    0    -1
+$EndComp
+Wire Wire Line
+	7600 5000 7600 4850
+Wire Wire Line
+	7600 4850 7850 4850
+Connection ~ 7850 4850
+Wire Wire Line
+	7850 5350 7600 5350
+Wire Wire Line
+	7600 5350 7600 5300
+Connection ~ 7850 5350
+Text Notes 1800 6500 0    60   ~ 0
+EN needs to be at least\n1.2v
+Text Notes 2500 2600 0    60   ~ 0
+NOTE: Update R when LED is picked out
+Text Notes 6700 4800 0    60   ~ 0
+Add a flyback diode?
 $EndSCHEMATC

Commit message: schematic nearing completion
Parts:
- added P?: +VBATT, symbol +VBATT
- added U?: ZXMHC6A07N8, symbol ZXMHC6A07N8
- R?: value R -> 1k
Connections:
- net labels added: WARN_LED_A, WARN_LED_B
- net labels removed: WARN_LED_EN, WARN_LED_SELECT
- wire segments 34 -> 51
Other:
- note added: "Conn to SMA"
- note added: "Using VBATT here is probably a bad idea"
Changed lines of the file:
@@
 Text HLabel 6850 5650 0    60   Input ~ 0
 PIEZO_OUT
-Text HLabel 9400 2400 2    60   Input ~ 0
-WARN_LED_SELECT
-Text HLabel 9400 2600 2    60   Input ~ 0
-WARN_LED_EN
+Text HLabel 7350 2400 0    60   Input ~ 0
+WARN_LED_A
+Text HLabel 7350 3550 0    60   Input ~ 0
+WARN_LED_B
 Text HLabel 1700 2800 0    60   Input ~ 0
 STATUS_LED
@@
 P 7300 5650
 F 0 "R?" V 7380 5650 50  0000 C CNN
-F 1 "R" V 7300 5650 50  0000 C CNN
+F 1 "1k" V 7300 5650 50  0000 C CNN
 F 2 "" V 7230 5650 30  0000 C CNN
 F 3 "" H 7300 5650 30  0000 C CNN
@@
 	1    0    0    -1
 $EndComp
-Wire Wire Line
-	2450 6200 2750 6200
-Wire Wire Line
-	7850 5200 7850 5450
-Wire Wire Line
-	7850 4750 7850 5100
-Wire Wire Line
-	7450 5650 7550 5650
-Wire Wire Line
-	7150 5650 6850 5650
-Wire Wire Line
-	1150 5800 1150 6000
-Wire Wire Line
-	1150 6000 2750 6000
-Wire Wire Line
-	1650 6050 1650 6000
-Connection ~ 1650 6000
-Wire Wire Line
-	1650 6750 1650 6350
-Wire Wire Line
-	2400 5450 2200 5450
-Wire Wire Line
-	2200 5450 2200 6000
-Connection ~ 2200 6000
-Wire Wire Line
-	3000 5450 3600 5450
-Wire Wire Line
-	3300 5700 3300 5450
-Connection ~ 3300 5450
-Wire Wire Line
-	4200 6200 4200 5900
-Wire Wire Line
-	3750 6100 4600 6100
-Connection ~ 4200 6100
-Wire Wire Line
-	4950 6700 1650 6700
-Wire Wire Line
-	3300 6700 3300 6550
-Connection ~ 1650 6700
-Wire Wire Line
-	4200 6700 4200 6500
-Connection ~ 3300 6700
-Wire Wire Line
-	4600 6100 4600 5900
-Wire Wire Line
-	3900 5450 5500 5450
-Wire Wire Line
-	4200 5450 4200 5600
-Wire Wire Line
-	4600 5450 4600 5600
-Connection ~ 4200 5450
-Wire Wire Line
-	4950 5450 4950 5600
-Connection ~ 4600 5450
-Wire Wire Line
-	4950 5900 4950 6700
-Connection ~ 4200 6700
-Wire Wire Line
-	5500 5450 5500 5350
-Connection ~ 4950 5450
-Wire Wire Line
-	7850 6050 7850 5850
 $Comp
 L LED D?
@@
 	1    0    0    -1
 $EndComp
-Wire Wire Line
-	1700 2800 1950 2800
-Wire Wire Line
-	2350 2800 2700 2800
-Wire Wire Line
-	3000 2800 3400 2800
-Wire Wire Line
-	3400 2800 3400 3000
 $Comp
 L R 1k
@@
 	1    0    0    -1
 $EndComp
-Wire Wire Line
-	7600 5000 7600 4850
-Wire Wire Line
-	7600 4850 7850 4850
-Connection ~ 7850 4850
-Wire Wire Line
-	7850 5350 7600 5350
-Wire Wire Line
-	7600 5350 7600 5300
-Connection ~ 7850 5350
 Text Notes 1800 6500 0    60   ~ 0
 EN needs to be at least\n1.2v
@@
 Text Notes 6700 4800 0    60   ~ 0
 Add a flyback diode?
+$Comp
+L ZXMHC6A07N8 U?
+U 1 1 553EC5C4
+P 8350 3050
+F 0 "U?" H 8220 3300 60  0000 C CNN
+F 1 "ZXMHC6A07N8" H 8720 2790 60  0000 C CNN
+F 2 "" H 8480 2900 60  0000 C CNN
+F 3 "" H 8480 2900 60  0000 C CNN
+	1    8350 3050
+	1    0    0    -1
+$EndComp
+$Comp
+L +VBATT P?
+U 1 1 553ECE83
+P 8350 1900
+F 0 "P?" H 8450 1900 60  0001 C CNN
+F 1 "+VBATT" H 8350 2200 60  0000 C CNN
+F 2 "" H 8350 1900 60  0000 C CNN
+F 3 "" H 8350 1900 60  0000 C CNN
+	1    8350 1900
+	1    0    0    -1
+$EndComp
+$Comp
+L GND #PWR?
+U 1 1 553ECF4B
+P 8350 3700
+F 0 "#PWR?" H 8350 3450 50  0001 C CNN
+F 1 "GND" H 8350 3550 50  0000 C CNN
+F 2 "" H 8350 3700 60  0000 C CNN
+F 3 "" H 8350 3700 60  0000 C CNN
+	1    8350 3700
+	1    0    0    -1
+$EndComp
+Wire Wire Line
+	2450 6200 2750 6200
+Wire Wire Line
+	7850 5200 7850 5450
+Wire Wire Line
+	7850 4750 7850 5100
+Wire Wire Line
+	7450 5650 7550 5650
+Wire Wire Line
+	7150 5650 6850 5650
+Wire Wire Line
+	1150 5800 1150 6000
+Wire Wire Line
+	1150 6000 2750 6000
+Wire Wire Line
+	1650 6050 1650 6000
+Connection ~ 1650 6000
+Wire Wire Line
+	1650 6750 1650 6350
+Wire Wire Line
+	2400 5450 2200 5450
+Wire Wire Line
+	2200 5450 2200 6000
+Connection ~ 2200 6000
+Wire Wire Line
+	3000 5450 3600 5450
+Wire Wire Line
+	3300 5700 3300 5450
+Connection ~ 3300 5450
+Wire Wire Line
+	4200 6200 4200 5900
+Wire Wire Line
+	3750 6100 4600 6100
+Connection ~ 4200 6100
+Wire Wire Line
+	4950 6700 1650 6700
+Wire Wire Line
+	3300 6700 3300 6550
+Connection ~ 1650 6700
+Wire Wire Line
+	4200 6700 4200 6500
+Connection ~ 3300 6700
+Wire Wire Line
+	4600 6100 4600 5900
+Wire Wire Line
+	3900 5450 5500 5450
+Wire Wire Line
+	4200 5450 4200 5600
+Wire Wire Line
+	4600 5450 4600 5600
+Connection ~ 4200 5450
+Wire Wire Line
+	4950 5450 4950 5600
+Connection ~ 4600 5450
+Wire Wire Line
+	4950 5900 4950 6700
+Connection ~ 4200 6700
+Wire Wire Line
+	5500 5450 5500 5350
+Connection ~ 4950 5450
+Wire Wire Line
+	7850 6050 7850 5850
+Wire Wire Line
+	1700 2800 1950 2800
+Wire Wire Line
+	2350 2800 2700 2800
+Wire Wire Line
+	3000 2800 3400 2800
+Wire Wire Line
+	3400 2800 3400 3000
+Wire Wire Line
+	7600 5000 7600 4850
+Wire Wire Line
+	7600 4850 7850 4850
+Connection ~ 7850 4850
+Wire Wire Line
+	7850 5350 7600 5350
+Wire Wire Line
+	7600 5350 7600 5300
+Connection ~ 7850 5350
+Wire Wire Line
+	8350 3700 8350 3450
+Wire Wire Line
+	8350 1900 8350 2650
+Wire Wire Line
+	7350 2400 9000 2400
+Wire Wire Line
+	9000 2400 9000 3150
+Wire Wire Line
+	9000 3150 8700 3150
+Wire Wire Line
+	8700 2950 9000 2950
+Wire Wire Line
+	9000 2950 9000 2900
+Connection ~ 9000 2900
+Wire Wire Line
+	7350 3550 7750 3550
+Wire Wire Line
+	7750 3550 7750 2950
+Wire Wire Line
+	7750 2950 8000 2950
+Wire Wire Line
+	8000 3150 7750 3150
+Connection ~ 7750 3150
+Wire Wire Line
+	8000 3050 7900 3050
+Wire Wire Line
+	7900 3050 7900 2550
+Wire Wire Line
+	7900 2550 9650 2550
+Wire Wire Line
+	8700 3050 9200 3050
+Wire Wire Line
+	9200 3050 9200 2650
+Wire Wire Line
+	9200 2650 9650 2650
+Text Notes 8650 1850 0    60   ~ 0
+Using VBATT here is probably a bad idea
+Text Notes 9800 2600 0    60   ~ 0
+Conn to SMA
 $EndSCHEMATC

Commit message: Added component values
Parts:
- D?: footprint (none) -> 0603
- R?: value R -> 120
Changed lines of the file:
@@
 F 0 "D?" H 2150 2900 50  0000 C CNN
 F 1 "LED" H 2150 2700 50  0000 C CNN
-F 2 "" H 2150 2800 60  0000 C CNN
+F 2 "0603" H 2300 2650 60  0000 C CNN
 F 3 "" H 2150 2800 60  0000 C CNN
 	1    2150 2800
-	-1   0    0    1
+	1    0    0    -1
 $EndComp
 $Comp
@@
 P 2850 2800
 F 0 "R?" V 2930 2800 50  0000 C CNN
-F 1 "R" V 2850 2800 50  0000 C CNN
+F 1 "120" V 2850 2800 50  0000 C CNN
 F 2 "" V 2780 2800 30  0000 C CNN
 F 3 "" H 2850 2800 30  0000 C CNN
@@
 	7850 6050 7850 5850
 Wire Wire Line
-	1700 2800 1950 2800
-Wire Wire Line
-	2350 2800 2700 2800
-Wire Wire Line
 	3000 2800 3400 2800
 Wire Wire Line
@@
 Text Notes 9800 2600 0    60   ~ 0
 Conn to SMA
+Wire Wire Line
+	1700 2800 1950 2800
+Wire Wire Line
+	2350 2800 2700 2800
 $EndSCHEMATC

Commit message: more changes
Parts:
- added CON2: MMCX_CONN, symbol MMCX_CONN
- D2: renamed from D?; footprint 0603 -> (none)
- gave numbers to parts that had none: 9
- renumbered 4.7u to U11, 10u to U12, 2.2m to U14, 130k to U15, 22p to U16, 1u to U17, 1k to U18
Other:
- note removed: "Conn to SMA"
Changed lines of the file:
@@
 STATUS_LED
 $Comp
-L TPS61041 U?
+L TPS61041 U13
 U 1 1 55366BB2
 P 3200 6200
-F 0 "U?" H 3050 6550 60  0000 C CNN
+F 0 "U13" H 3050 6550 60  0000 C CNN
 F 1 "TPS61041" H 3550 6000 60  0000 C CNN
 F 2 "" H 3200 6200 60  0000 C CNN
@@
 $EndComp
 $Comp
-L PIEZO C?
+L PIEZO C30
 U 1 1 55381327
 P 8150 5150
-F 0 "C?" H 8100 5350 60  0000 C CNN
+F 0 "C30" H 8100 5350 60  0000 C CNN
 F 1 "PIEZO" H 8250 4950 60  0000 C CNN
 F 2 "" H 8150 5150 60  0000 C CNN
@@
 $EndComp
 $Comp
-L Q_NPN_BCE Q?
+L Q_NPN_BCE Q1
 U 1 1 5538136D
 P 7750 5650
-F 0 "Q?" H 8050 5700 50  0000 R CNN
+F 0 "Q1" H 8050 5700 50  0000 R CNN
 F 1 "Q_NPN_BCE" H 8350 5600 50  0000 R CNN
 F 2 "" H 7950 5750 29  0000 C CNN
@@
 $EndComp
 $Comp
-L +24V #PWR?
+L +24V #PWR52
 U 1 1 553813E6
 P 7850 4750
-F 0 "#PWR?" H 7850 4600 50  0001 C CNN
+F 0 "#PWR52" H 7850 4600 50  0001 C CNN
 F 1 "+24V" H 7850 4890 50  0000 C CNN
 F 2 "" H 7850 4750 60  0000 C CNN
@@
 $EndComp
 $Comp
-L R R?
+L R R12
 U 1 1 55381462
 P 7300 5650
-F 0 "R?" V 7380 5650 50  0000 C CNN
+F 0 "R12" V 7380 5650 50  0000 C CNN
 F 1 "1k" V 7300 5650 50  0000 C CNN
 F 2 "" V 7230 5650 30  0000 C CNN
@@
 $EndComp
 $Comp
-L C 4.7u
+L C U11
 U 1 1 55381689
 P 1650 6200
-F 0 "4.7u" H 1675 6300 50  0000 L CNN
+F 0 "U11" H 1675 6300 50  0000 L CNN
 F 1 "C" H 1675 6100 50  0000 L CNN
 F 2 "" H 1688 6050 30  0000 C CNN
@@
 $EndComp
 $Comp
-L +VBATT P?
+L +VBATT P2
 U 1 1 553816AE
 P 1150 5800
-F 0 "P?" H 1250 5800 60  0001 C CNN
+F 0 "P2" H 1250 5800 60  0001 C CNN
 F 1 "+VBATT" H 1150 6100 60  0000 C CNN
 F 2 "" H 1150 5800 60  0000 C CNN
@@
 $EndComp
 $Comp
-L GND #PWR?
+L GND #PWR49
 U 1 1 55381751
 P 1650 6750
-F 0 "#PWR?" H 1650 6500 50  0001 C CNN
+F 0 "#PWR49" H 1650 6500 50  0001 C CNN
 F 1 "GND" H 1650 6600 50  0000 C CNN
 F 2 "" H 1650 6750 60  0000 C CNN
@@
 $EndComp
 $Comp
-L INDUCTOR 10u
+L INDUCTOR U12
 U 1 1 553817A7
 P 2700 5450
-F 0 "10u" V 2650 5450 50  0000 C CNN
+F 0 "U12" V 2650 5450 50  0000 C CNN
 F 1 "INDUCTOR" V 2800 5450 50  0000 C CNN
 F 2 "" H 2700 5450 60  0000 C CNN
@@
 $EndComp
 $Comp
-L D_Schottky D?
+L D_Schottky D3
 U 1 1 55381819
 P 3750 5450
-F 0 "D?" H 3750 5550 50  0000 C CNN
+F 0 "D3" H 3750 5550 50  0000 C CNN
 F 1 "D_Schottky" H 3750 5350 50  0000 C CNN
 F 2 "" H 3750 5450 60  0000 C CNN
@@
 $EndComp
 $Comp
-L R 2.2m
+L R U14
 U 1 1 55381851
 P 4200 5750
-F 0 "2.2m" V 4280 5750 50  0000 C CNN
+F 0 "U14" V 4280 5750 50  0000 C CNN
 F 1 "R" V 4200 5750 50  0000 C CNN
 F 2 "" V 4130 5750 30  0000 C CNN
@@
 $EndComp
 $Comp
-L R 130k
+L R U15
 U 1 1 5538187A
 P 4200 6350
-F 0 "130k" V 4280 6350 50  0000 C CNN
+F 0 "U15" V 4280 6350 50  0000 C CNN
 F 1 "R" V 4200 6350 50  0000 C CNN
 F 2 "" V 4130 6350 30  0000 C CNN
@@
 $EndComp
 $Comp
-L C 22p
+L C U16
 U 1 1 553818B9
 P 4600 5750
-F 0 "22p" H 4625 5850 50  0000 L CNN
+F 0 "U16" H 4625 5850 50  0000 L CNN
 F 1 "C" H 4625 5650 50  0000 L CNN
 F 2 "" H 4638 5600 30  0000 C CNN
@@
 $EndComp
 $Comp
-L C 1u
+L C U17
 U 1 1 553818E7
 P 4950 5750
-F 0 "1u" H 4975 5850 50  0000 L CNN
+F 0 "U17" H 4975 5850 50  0000 L CNN
 F 1 "C" H 4975 5650 50  0000 L CNN
 F 2 "" H 4988 5600 30  0000 C CNN
@@
 $EndComp
 $Comp
-L +24V #PWR?
+L +24V #PWR51
 U 1 1 55381C1E
 P 5500 5350
-F 0 "#PWR?" H 5500 5200 50  0001 C CNN
+F 0 "#PWR51" H 5500 5200 50  0001 C CNN
 F 1 "+24V" H 5500 5490 50  0000 C CNN
 F 2 "" H 5500 5350 60  0000 C CNN
@@
 $EndComp
 $Comp
-L GND #PWR?
+L GND #PWR53
 U 1 1 55381CB8
 P 7850 6050
-F 0 "#PWR?" H 7850 5800 50  0001 C CNN
+F 0 "#PWR53" H 7850 5800 50  0001 C CNN
 F 1 "GND" H 7850 5900 50  0000 C CNN
 F 2 "" H 7850 6050 60  0000 C CNN
@@
 $EndComp
 $Comp
-L LED D?
+L LED D2
 U 1 1 55381AF7
 P 2150 2800
-F 0 "D?" H 2150 2900 50  0000 C CNN
+F 0 "D2" H 2150 2900 50  0000 C CNN
 F 1 "LED" H 2150 2700 50  0000 C CNN
-F 2 "0603" H 2300 2650 60  0000 C CNN
+F 2 "" H 2300 2650 60  0000 C CNN
 F 3 "" H 2150 2800 60  0000 C CNN
 	1    2150 2800
@@
 $EndComp
 $Comp
-L R R?
+L R R11
 U 1 1 55381B8F
 P 2850 2800
-F 0 "R?" V 2930 2800 50  0000 C CNN
+F 0 "R11" V 2930 2800 50  0000 C CNN
 F 1 "120" V 2850 2800 50  0000 C CNN
 F 2 "" V 2780 2800 30  0000 C CNN
@@
 $EndComp
 $Comp
-L GND #PWR?
+L GND #PWR50
 U 1 1 55381C08
 P 3400 3000
-F 0 "#PWR?" H 3400 2750 50  0001 C CNN
+F 0 "#PWR50" H 3400 2750 50  0001 C CNN
 F 1 "GND" H 3400 2850 50  0000 C CNN
 F 2 "" H 3400 3000 60  0000 C CNN
@@
 $EndComp
 $Comp
-L R 1k
+L R U18
 U 1 1 55387943
 P 7600 5150
-F 0 "1k" V 7680 5150 50  0000 C CNN
+F 0 "U18" V 7680 5150 50  0000 C CNN
 F 1 "R" V 7600 5150 50  0000 C CNN
 F 2 "" V 7530 5150 30  0000 C CNN
@@
 Add a flyback diode?
 $Comp
-L ZXMHC6A07N8 U?
+L ZXMHC6A07N8 U19
 U 1 1 553EC5C4
 P 8350 3050
-F 0 "U?" H 8220 3300 60  0000 C CNN
+F 0 "U19" H 8220 3300 60  0000 C CNN
 F 1 "ZXMHC6A07N8" H 8720 2790 60  0000 C CNN
 F 2 "" H 8480 2900 60  0000 C CNN
@@
 $EndComp
 $Comp
-L +VBATT P?
+L +VBATT P3
 U 1 1 553ECE83
 P 8350 1900
-F 0 "P?" H 8450 1900 60  0001 C CNN
+F 0 "P3" H 8450 1900 60  0001 C CNN
 F 1 "+VBATT" H 8350 2200 60  0000 C CNN
 F 2 "" H 8350 1900 60  0000 C CNN
@@
 $EndComp
 $Comp
-L GND #PWR?
+L GND #PWR54
 U 1 1 553ECF4B
 P 8350 3700
-F 0 "#PWR?" H 8350 3450 50  0001 C CNN
+F 0 "#PWR54" H 8350 3450 50  0001 C CNN
 F 1 "GND" H 8350 3550 50  0000 C CNN
 F 2 "" H 8350 3700 60  0000 C CNN
@@
 	1    0    0    -1
 $EndComp
+Text Notes 8650 1850 0    60   ~ 0
+Using VBATT here is probably a bad idea
 Wire Wire Line
 	2450 6200 2750 6200
@@
 	7900 3050 7900 2550
 Wire Wire Line
-	7900 2550 9650 2550
+	7900 2550 9750 2550
 Wire Wire Line
 	8700 3050 9200 3050
@@
 	9200 3050 9200 2650
 Wire Wire Line
-	9200 2650 9650 2650
-Text Notes 8650 1850 0    60   ~ 0
-Using VBATT here is probably a bad idea
-Text Notes 9800 2600 0    60   ~ 0
-Conn to SMA
+	9200 2650 9750 2650
 Wire Wire Line
 	1700 2800 1950 2800
 Wire Wire Line
 	2350 2800 2700 2800
+$Comp
+L MMCX_CONN CON2
+U 1 1 5540F4C0
+P 9900 2650
+F 0 "CON2" H 10100 2850 60  0000 C CNN
+F 1 "MMCX_CONN" H 10050 2500 60  0000 C CNN
+F 2 "" H 9900 2650 60  0000 C CNN
+F 3 "" H 9900 2650 60  0000 C CNN
+	1    9900 2650
+	1    0    0    -1
+$EndComp
 $EndSCHEMATC

Commit message: mega commit
Parts:
- removed C30: PIEZO, symbol PIEZO
- removed P2, P3: +VBATT, symbol +VBATT
- removed Q1: Q_NPN_BCE, symbol Q_NPN_BCE
- added AUD1: PIEZO, aero:Piezo_Solder_Conn, symbol PIEZO
- added Q1: Q_NPN_BEC, Housings_SOT-23_SOT-143_TSOT-6:SOT-23, symbol Q_NPN_BEC
- C32: renamed from U11; value C -> 4.7uF; footprint (none) -> Capacitors_SMD:C_0603
- C33: renamed from U16; value C -> 22pF; footprint (none) -> Capacitors_SMD:C_0603
- C34: renamed from U17; value C -> 100nF; footprint (none) -> Capacitors_SMD:C_0603
- CON2: footprint (none) -> aero:CONMMCX002-SMD
- D2: footprint (none) -> LEDs:LED-0805
- D3: footprint (none) -> Diodes_SMD:SOD-123
- L4: renamed from U12; value INDUCTOR -> 10u; footprint (none) -> aero:SDR0703; Part# (none) -> LQH3C100K24
- R12: renamed from R11; footprint (none) -> Resistors_SMD:R_0603
- R13: renamed from U14; value R -> 2.21m; footprint (none) -> Resistors_SMD:R_0603
- R14: renamed from U15; value R -> 140k; footprint (none) -> Resistors_SMD:R_0603
- R15: renamed from R12; value 1k -> 3k; footprint (none) -> Resistors_SMD:R_0603
- R16: renamed from U18; value R -> 2k; footprint (none) -> Resistors_SMD:R_0603
- U8: renamed from U13; footprint (none) -> Housings_SOT-23_SOT-143_TSOT-6:SOT-23-5
- U9: renamed from U19; footprint (none) -> Power_Integrations:SO-8
Connections:
- net labels added: +VBATT
- wire segments 51 -> 52
Other:
- note added: "Confirm pin assignments of NPN"

Commit message: Finished layout
Changed lines of the file:
@@
 EESchema Schematic File Version 2
+LIBS:aero-rescue
 LIBS:aero
 LIBS:power
@@
 LIBS:memory
 LIBS:xilinx
-LIBS:special
 LIBS:microcontrollers
 LIBS:dsp
@@
 $EndComp
 $Comp
-L +24V #PWR053
+L +24V-RESCUE-aero #PWR053
 U 1 1 553813E6
 P 7850 4750
+AR Path="/553813E6" Ref="#PWR053"  Part="1"
+AR Path="/55359120/553813E6" Ref="#PWR053"  Part="1"
 F 0 "#PWR053" H 7850 4600 50  0001 C CNN
 F 1 "+24V" H 7850 4890 50  0000 C CNN
@@
 F 3 "" H 3750 5450 60  0000 C CNN
 	1    3750 5450
-	1    0    0    -1
+	-1   0    0    1
 $EndComp
 $Comp
@@
 $EndComp
 $Comp
-L +24V #PWR056
+L +24V-RESCUE-aero #PWR056
 U 1 1 55381C1E
 P 5500 5350
+AR Path="/55381C1E" Ref="#PWR056"  Part="1"
+AR Path="/55359120/55381C1E" Ref="#PWR056"  Part="1"
 F 0 "#PWR056" H 5500 5200 50  0001 C CNN
 F 1 "+24V" H 5500 5490 50  0000 C CNN

Commit message: hw fixes
Parts:
- Q1: symbol Q_NPN_BEC -> Q_NPN_BEC-RESCUE-aero
Changed lines of the file:
@@
 Confirm pin assignments of NPN
 $Comp
-L Q_NPN_BEC Q1
+L Q_NPN_BEC-RESCUE-aero Q1
 U 1 1 5546CD30
 P 7750 5650

Commit message: committing hardware updates (probably unnecessary)
Parts:
- R16: value 2k -> 3k
Changed lines of the file:
@@
 P 7600 5150
 F 0 "R16" V 7680 5150 50  0000 C CNN
-F 1 "2k" V 7600 5150 50  0000 C CNN
+F 1 "3k" V 7600 5150 50  0000 C CNN
 F 2 "Resistors_SMD:R_0603" V 7530 5150 30  0001 C CNN
 F 3 "" H 7600 5150 30  0000 C CNN
@@
 Text Notes 2500 2600 0    60   ~ 0
 NOTE: Update R when LED is picked out
-Text Notes 8700 6250 0    60   ~ 0
+Text Notes 8950 6250 0    60   ~ 0
 Add a flyback diode?
 $Comp
@@
 	1    0    0    -1
 $EndComp
-Text Notes 8050 6050 0    60   ~ 0
+Text Notes 8750 6000 0    60   ~ 0
 Confirm pin assignments of NPN
 $Comp
