File: hardware/pcb/bmx055.sch (KiCad schematic (older format))
At the start: 3 parts, among them U3 BMX055

Commit message: more changes
Parts:
- U5, U6: renamed from 100nF; value C -> 100nF
- renumbered U3 to U4
Changed lines of the file:
@@
 $EndDescr
 $Comp
-L BMX055 U3
+L BMX055 U4
 U 1 1 5527EBA6
 P 5600 3000
-F 0 "U3" H 5900 2150 60  0000 C CNN
+F 0 "U4" H 5900 2150 60  0000 C CNN
 F 1 "BMX055" H 5150 2150 60  0000 C CNN
 F 2 "aero:BMX055" H 5600 3000 60  0001 C CNN
@@
 NoConn ~ 6150 3550
 $Comp
-L +3V #PWR028
+L +3V #PWR36
 U 1 1 552EACA4
 P 6900 2000
-F 0 "#PWR028" H 6900 1900 60  0001 C CNN
+F 0 "#PWR36" H 6900 1900 60  0001 C CNN
 F 1 "+3V" H 6750 2150 60  0000 C CNN
 F 2 "" H 6900 2000 60  0000 C CNN
@@
 $EndComp
 $Comp
-L GND #PWR029
+L GND #PWR37
 U 1 1 552EACBF
 P 6900 4050
-F 0 "#PWR029" H 6900 3800 50  0001 C CNN
+F 0 "#PWR37" H 6900 3800 50  0001 C CNN
 F 1 "GND" H 6900 3900 50  0000 C CNN
 F 2 "" H 6900 4050 60  0000 C CNN
@@
 $EndComp
 $Comp
-L GND #PWR030
+L GND #PWR35
 U 1 1 552EACD5
 P 4500 4100
-F 0 "#PWR030" H 4500 3850 50  0001 C CNN
+F 0 "#PWR35" H 4500 3850 50  0001 C CNN
 F 1 "GND" H 4500 3950 50  0000 C CNN
 F 2 "" H 4500 4100 60  0000 C CNN
@@
 	6900 2950 6900 4050
 $Comp
-L +3V #PWR031
+L +3V #PWR38
 U 1 1 552EBBB1
 P 7900 2450
-F 0 "#PWR031" H 7900 2350 60  0001 C CNN
+F 0 "#PWR38" H 7900 2350 60  0001 C CNN
 F 1 "+3V" H 7750 2600 60  0000 C CNN
 F 2 "" H 7900 2450 60  0000 C CNN
@@
 $EndComp
 $Comp
-L GND #PWR032
+L GND #PWR39
 U 1 1 552EBBC7
 P 7900 3050
-F 0 "#PWR032" H 7900 2800 50  0001 C CNN
+F 0 "#PWR39" H 7900 2800 50  0001 C CNN
 F 1 "GND" H 7900 2900 50  0000 C CNN
 F 2 "" H 7900 3050 60  0000 C CNN
@@
 $EndComp
 $Comp
-L C 100nF
+L C U5
 U 1 1 552EBBDD
 P 7700 2750
-F 0 "100nF" H 7725 2850 50  0000 L CNN
-F 1 "C" H 7725 2650 50  0000 L CNN
+F 0 "U5" H 7725 2850 50  0000 L CNN
+F 1 "100nF" H 7725 2650 50  0000 L CNN
 F 2 "" H 7738 2600 30  0000 C CNN
 F 3 "" H 7700 2750 60  0000 C CNN
@@
 $EndComp
 $Comp
-L C 100nF
+L C U6
 U 1 1 552EBBFD
 P 8050 2750
-F 0 "100nF" H 8075 2850 50  0000 L CNN
-F 1 "C" H 8075 2650 50  0000 L CNN
+F 0 "U6" H 8075 2850 50  0000 L CNN
+F 1 "100nF" H 8075 2650 50  0000 L CNN
 F 2 "" H 8088 2600 30  0000 C CNN
 F 3 "" H 8050 2750 60  0000 C CNN

Commit message: mega commit
Parts:
- C25: renamed from U5; footprint (none) -> Capacitors_SMD:C_0603
- C26: renamed from U6; footprint (none) -> Capacitors_SMD:C_0603
Changed lines of the file:
@@
 NoConn ~ 6150 3550
 $Comp
-L +3V #PWR36
+L +3V #PWR036
 U 1 1 552EACA4
 P 6900 2000
-F 0 "#PWR36" H 6900 1900 60  0001 C CNN
+F 0 "#PWR036" H 6900 1900 60  0001 C CNN
 F 1 "+3V" H 6750 2150 60  0000 C CNN
 F 2 "" H 6900 2000 60  0000 C CNN
@@
 $EndComp
 $Comp
-L GND #PWR37
+L GND #PWR037
 U 1 1 552EACBF
 P 6900 4050
-F 0 "#PWR37" H 6900 3800 50  0001 C CNN
+F 0 "#PWR037" H 6900 3800 50  0001 C CNN
 F 1 "GND" H 6900 3900 50  0000 C CNN
 F 2 "" H 6900 4050 60  0000 C CNN
@@
 $EndComp
 $Comp
-L GND #PWR35
+L GND #PWR038
 U 1 1 552EACD5
 P 4500 4100
-F 0 "#PWR35" H 4500 3850 50  0001 C CNN
+F 0 "#PWR038" H 4500 3850 50  0001 C CNN
 F 1 "GND" H 4500 3950 50  0000 C CNN
 F 2 "" H 4500 4100 60  0000 C CNN
@@
 	6900 2950 6900 4050
 $Comp
-L +3V #PWR38
+L +3V #PWR039
 U 1 1 552EBBB1
 P 7900 2450
-F 0 "#PWR38" H 7900 2350 60  0001 C CNN
+F 0 "#PWR039" H 7900 2350 60  0001 C CNN
 F 1 "+3V" H 7750 2600 60  0000 C CNN
 F 2 "" H 7900 2450 60  0000 C CNN
@@
 $EndComp
 $Comp
-L GND #PWR39
+L GND #PWR040
 U 1 1 552EBBC7
 P 7900 3050
-F 0 "#PWR39" H 7900 2800 50  0001 C CNN
+F 0 "#PWR040" H 7900 2800 50  0001 C CNN
 F 1 "GND" H 7900 2900 50  0000 C CNN
 F 2 "" H 7900 3050 60  0000 C CNN
@@
 $EndComp
 $Comp
-L C U5
+L C C25
 U 1 1 552EBBDD
 P 7700 2750
-F 0 "U5" H 7725 2850 50  0000 L CNN
+F 0 "C25" H 7725 2850 50  0000 L CNN
 F 1 "100nF" H 7725 2650 50  0000 L CNN
-F 2 "" H 7738 2600 30  0000 C CNN
+F 2 "Capacitors_SMD:C_0603" H 7738 2600 30  0001 C CNN
 F 3 "" H 7700 2750 60  0000 C CNN
 	1    7700 2750
@@
 $EndComp
 $Comp
-L C U6
+L C C26
 U 1 1 552EBBFD
 P 8050 2750
-F 0 "U6" H 8075 2850 50  0000 L CNN
+F 0 "C26" H 8075 2850 50  0000 L CNN
 F 1 "100nF" H 8075 2650 50  0000 L CNN
-F 2 "" H 8088 2600 30  0000 C CNN
+F 2 "Capacitors_SMD:C_0603" H 8088 2600 30  0001 C CNN
 F 3 "" H 8050 2750 60  0000 C CNN
 	1    8050 2750

Commit message: pre major restructuring commit
Parts:
- C22: renamed from C25; footprint Capacitors_SMD:C_0603 -> Capacitors_SMD:C_0402
- C23: renamed from C26; footprint Capacitors_SMD:C_0603 -> Capacitors_SMD:C_0402
- renumbered U4 to U5
Changed lines of the file:
@@
 $Descr A4 11693 8268
 encoding utf-8
-Sheet 4 7
+Sheet 4 8
 Title ""
 Date ""
@@
 $EndDescr
 $Comp
-L BMX055 U4
+L BMX055 U5
 U 1 1 5527EBA6
 P 5600 3000
-F 0 "U4" H 5900 2150 60  0000 C CNN
+F 0 "U5" H 5900 2150 60  0000 C CNN
 F 1 "BMX055" H 5150 2150 60  0000 C CNN
 F 2 "aero:BMX055" H 5600 3000 60  0001 C CNN
@@
 NoConn ~ 6150 3550
 $Comp
-L +3V #PWR036
+L +3V #PWR032
 U 1 1 552EACA4
 P 6900 2000
-F 0 "#PWR036" H 6900 1900 60  0001 C CNN
+F 0 "#PWR032" H 6900 1900 60  0001 C CNN
 F 1 "+3V" H 6750 2150 60  0000 C CNN
 F 2 "" H 6900 2000 60  0000 C CNN
@@
 $EndComp
 $Comp
-L GND #PWR037
+L GND #PWR033
 U 1 1 552EACBF
 P 6900 4050
-F 0 "#PWR037" H 6900 3800 50  0001 C CNN
+F 0 "#PWR033" H 6900 3800 50  0001 C CNN
 F 1 "GND" H 6900 3900 50  0000 C CNN
 F 2 "" H 6900 4050 60  0000 C CNN
@@
 $EndComp
 $Comp
-L GND #PWR038
+L GND #PWR034
 U 1 1 552EACD5
 P 4500 4100
-F 0 "#PWR038" H 4500 3850 50  0001 C CNN
+F 0 "#PWR034" H 4500 3850 50  0001 C CNN
 F 1 "GND" H 4500 3950 50  0000 C CNN
 F 2 "" H 4500 4100 60  0000 C CNN
@@
 	6900 2950 6900 4050
 $Comp
-L +3V #PWR039
+L +3V #PWR035
 U 1 1 552EBBB1
 P 7900 2450
-F 0 "#PWR039" H 7900 2350 60  0001 C CNN
+F 0 "#PWR035" H 7900 2350 60  0001 C CNN
 F 1 "+3V" H 7750 2600 60  0000 C CNN
 F 2 "" H 7900 2450 60  0000 C CNN
@@
 $EndComp
 $Comp
-L GND #PWR040
+L GND #PWR036
 U 1 1 552EBBC7
 P 7900 3050
-F 0 "#PWR040" H 7900 2800 50  0001 C CNN
+F 0 "#PWR036" H 7900 2800 50  0001 C CNN
 F 1 "GND" H 7900 2900 50  0000 C CNN
 F 2 "" H 7900 3050 60  0000 C CNN
@@
 $EndComp
 $Comp
-L C C25
+L C C22
 U 1 1 552EBBDD
 P 7700 2750
-F 0 "C25" H 7725 2850 50  0000 L CNN
+F 0 "C22" H 7725 2850 50  0000 L CNN
 F 1 "100nF" H 7725 2650 50  0000 L CNN
-F 2 "Capacitors_SMD:C_0603" H 7738 2600 30  0001 C CNN
+F 2 "Capacitors_SMD:C_0402" H 7738 2600 30  0001 C CNN
 F 3 "" H 7700 2750 60  0000 C CNN
 	1    7700 2750
@@
 $EndComp
 $Comp
-L C C26
+L C C23
 U 1 1 552EBBFD
 P 8050 2750
-F 0 "C26" H 8075 2850 50  0000 L CNN
+F 0 "C23" H 8075 2850 50  0000 L CNN
 F 1 "100nF" H 8075 2650 50  0000 L CNN
-F 2 "Capacitors_SMD:C_0603" H 8088 2600 30  0001 C CNN
+F 2 "Capacitors_SMD:C_0402" H 8088 2600 30  0001 C CNN
 F 3 "" H 8050 2750 60  0000 C CNN
 	1    8050 2750

Commit message: more progress on new layout
Parts:
- renumbered C22 to C20, C23 to C21
Changed lines of the file:
@@
 $EndComp
 $Comp
-L C C22
+L C C20
 U 1 1 552EBBDD
 P 7700 2750
-F 0 "C22" H 7725 2850 50  0000 L CNN
+F 0 "C20" H 7725 2850 50  0000 L CNN
 F 1 "100nF" H 7725 2650 50  0000 L CNN
 F 2 "Capacitors_SMD:C_0402" H 7738 2600 30  0001 C CNN
@@
 $EndComp
 $Comp
-L C C23
+L C C21
 U 1 1 552EBBFD
 P 8050 2750
-F 0 "C23" H 8075 2850 50  0000 L CNN
+F 0 "C21" H 8075 2850 50  0000 L CNN
 F 1 "100nF" H 8075 2650 50  0000 L CNN
 F 2 "Capacitors_SMD:C_0402" H 8088 2600 30  0001 C CNN
