File: hardware/pcb/ms5611.sch (KiCad schematic (older format))
At the start: 2 parts, among them U2 ms5611

Commit message: Added component values
Parts:
- C14: value C -> 100nF
Changed lines of the file:
@@
 P 4500 3700
 F 0 "C14" H 4525 3800 50  0000 L CNN
-F 1 "C" H 4525 3600 50  0000 L CNN
+F 1 "100nF" H 4525 3600 50  0000 L CNN
 F 2 "Capacitors_SMD:C_0402" H 4538 3550 30  0001 C CNN
 F 3 "" H 4500 3700 60  0000 C CNN

Commit message: more changes
Parts:
- renumbered C14 to C24, U2 to U3
Changed lines of the file:
@@
 $EndDescr
 $Comp
-L ms5611 U2
+L ms5611 U3
 U 1 1 551EEE6D
 P 5350 3550
-F 0 "U2" H 5550 3350 60  0000 C CNN
+F 0 "U3" H 5550 3350 60  0000 C CNN
 F 1 "ms5611" H 5300 4000 60  0000 C CNN
 F 2 "aero:ms5611" H 5350 3550 60  0001 C CNN
@@
 $EndComp
 $Comp
-L C C14
+L C C24
 U 1 1 551EEEE9
 P 4500 3700
-F 0 "C14" H 4525 3800 50  0000 L CNN
+F 0 "C24" H 4525 3800 50  0000 L CNN
 F 1 "100nF" H 4525 3600 50  0000 L CNN
 F 2 "Capacitors_SMD:C_0402" H 4538 3550 30  0001 C CNN
@@
 $EndComp
 $Comp
-L GND #PWR026
+L GND #PWR33
 U 1 1 551EEF1B
 P 4350 3150
-F 0 "#PWR026" H 4350 2900 50  0001 C CNN
+F 0 "#PWR33" H 4350 2900 50  0001 C CNN
 F 1 "GND" H 4350 3000 50  0000 C CNN
 F 2 "" H 4350 3150 60  0000 C CNN
@@
 Connection ~ 4900 3250
 $Comp
-L +3V #PWR027
+L +3V #PWR34
 U 1 1 55281F01
 P 4350 4100
-F 0 "#PWR027" H 4350 4000 60  0001 C CNN
+F 0 "#PWR34" H 4350 4000 60  0001 C CNN
 F 1 "+3V" H 4200 4250 60  0000 C CNN
 F 2 "" H 4350 4100 60  0000 C CNN

Commit message: mega commit
Parts:
- C24: footprint Capacitors_SMD:C_0402 -> Capacitors_SMD:C_0603
Changed lines of the file:
@@
 F 0 "C24" H 4525 3800 50  0000 L CNN
 F 1 "100nF" H 4525 3600 50  0000 L CNN
-F 2 "Capacitors_SMD:C_0402" H 4538 3550 30  0001 C CNN
+F 2 "Capacitors_SMD:C_0603" H 4538 3550 30  0001 C CNN
 F 3 "" H 4500 3700 60  0000 C CNN
 	1    4500 3700
@@
 $EndComp
 $Comp
-L GND #PWR33
+L GND #PWR034
 U 1 1 551EEF1B
 P 4350 3150
-F 0 "#PWR33" H 4350 2900 50  0001 C CNN
+F 0 "#PWR034" H 4350 2900 50  0001 C CNN
 F 1 "GND" H 4350 3000 50  0000 C CNN
 F 2 "" H 4350 3150 60  0000 C CNN
@@
 Connection ~ 4900 3250
 $Comp
-L +3V #PWR34
+L +3V #PWR035
 U 1 1 55281F01
 P 4350 4100
-F 0 "#PWR34" H 4350 4000 60  0001 C CNN
+F 0 "#PWR035" H 4350 4000 60  0001 C CNN
 F 1 "+3V" H 4200 4250 60  0000 C CNN
 F 2 "" H 4350 4100 60  0000 C CNN

Commit message: pre major restructuring commit
Parts:
- C21: renamed from C24; footprint Capacitors_SMD:C_0603 -> Capacitors_SMD:C_0402
- renumbered U3 to U4
Changed lines of the file:
@@
 $Descr A4 11693 8268
 encoding utf-8
-Sheet 3 7
+Sheet 3 8
 Title ""
 Date ""
@@
 $EndDescr
 $Comp
-L ms5611 U3
+L ms5611 U4
 U 1 1 551EEE6D
 P 5350 3550
-F 0 "U3" H 5550 3350 60  0000 C CNN
+F 0 "U4" H 5550 3350 60  0000 C CNN
 F 1 "ms5611" H 5300 4000 60  0000 C CNN
 F 2 "aero:ms5611" H 5350 3550 60  0001 C CNN
@@
 $EndComp
 $Comp
-L C C24
+L C C21
 U 1 1 551EEEE9
 P 4500 3700
-F 0 "C24" H 4525 3800 50  0000 L CNN
+F 0 "C21" H 4525 3800 50  0000 L CNN
 F 1 "100nF" H 4525 3600 50  0000 L CNN
-F 2 "Capacitors_SMD:C_0603" H 4538 3550 30  0001 C CNN
+F 2 "Capacitors_SMD:C_0402" H 4538 3550 30  0001 C CNN
 F 3 "" H 4500 3700 60  0000 C CNN
 	1    4500 3700
@@
 $EndComp
 $Comp
-L GND #PWR034
+L GND #PWR030
 U 1 1 551EEF1B
 P 4350 3150
-F 0 "#PWR034" H 4350 2900 50  0001 C CNN
+F 0 "#PWR030" H 4350 2900 50  0001 C CNN
 F 1 "GND" H 4350 3000 50  0000 C CNN
 F 2 "" H 4350 3150 60  0000 C CNN
@@
 Connection ~ 4900 3250
 $Comp
-L +3V #PWR035
+L +3V #PWR031
 U 1 1 55281F01
 P 4350 4100
-F 0 "#PWR035" H 4350 4000 60  0001 C CNN
+F 0 "#PWR031" H 4350 4000 60  0001 C CNN
 F 1 "+3V" H 4200 4250 60  0000 C CNN
 F 2 "" H 4350 4100 60  0000 C CNN

Commit message: more progress on new layout
Parts:
- renumbered C21 to C19
Changed lines of the file:
@@
 $EndComp
 $Comp
-L C C21
+L C C19
 U 1 1 551EEEE9
 P 4500 3700
-F 0 "C21" H 4525 3800 50  0000 L CNN
+F 0 "C19" H 4525 3800 50  0000 L CNN
 F 1 "100nF" H 4525 3600 50  0000 L CNN
 F 2 "Capacitors_SMD:C_0402" H 4538 3550 30  0001 C CNN
