File: hardware/pcb/power.sch (KiCad schematic (older format))
At the start: 15 parts, among them CON1 USB-MICRO-B, J2 LiPoly_Conn, U7 BQ24040DSQ, U8 TPS783

Commit message: ver2 is nearing completion.
Parts:
- added C32: 100nF, Capacitors_SMD:C_0402, symbol C
- added R15, R16: 10m, Resistors_SMD:R_0402, symbol R
Connections:
- net GND: now also C32.1, R16.1
- net Vbatt: now also R15.2
- new net BATT_SENSE: C32.2, R15.1, R16.2
Changed lines of the file:
@@
 	5550 4000 5550 3650
 Wire Wire Line
-	5750 4150 5750 4000
+	5750 2075 5750 4150
 Connection ~ 5750 4000
 Wire Wire Line
@@
 Text Label 5150 5800 0    60   ~ 0
 http://www.molex.com/molex/products/datasheet.jsp?part=active/0781710002_PCB_HEADERS.xml#partdetail
+$Comp
+L R R15
+U 1 1 55C04C61
+P 7275 2075
+F 0 "R15" V 7355 2075 50  0000 C CNN
+F 1 "10m" V 7275 2075 50  0000 C CNN
+F 2 "Resistors_SMD:R_0402" V 7205 2075 30  0001 C CNN
+F 3 "" H 7275 2075 30  0000 C CNN
+	1    7275 2075
+	0    1    1    0
+$EndComp
+$Comp
+L R R16
+U 1 1 55C04CB8
+P 7950 2075
+F 0 "R16" V 8030 2075 50  0000 C CNN
+F 1 "10m" V 7950 2075 50  0000 C CNN
+F 2 "Resistors_SMD:R_0402" V 7880 2075 30  0001 C CNN
+F 3 "" H 7950 2075 30  0000 C CNN
+	1    7950 2075
+	0    1    1    0
+$EndComp
+$Comp
+L GND #PWR049
+U 1 1 55C04D3B
+P 8350 2425
+F 0 "#PWR049" H 8350 2175 50  0001 C CNN
+F 1 "GND" H 8350 2275 50  0000 C CNN
+F 2 "" H 8350 2425 60  0000 C CNN
+F 3 "" H 8350 2425 60  0000 C CNN
+	1    8350 2425
+	1    0    0    -1
+$EndComp
+Text HLabel 8175 1475 2    60   Input ~ 0
+BATT_SENSE
+$Comp
+L C C32
+U 1 1 55C0577C
+P 7975 1750
+F 0 "C32" H 8000 1850 50  0000 L CNN
+F 1 "100nF" H 8000 1650 50  0000 L CNN
+F 2 "Capacitors_SMD:C_0402" H 8013 1600 30  0001 C CNN
+F 3 "" H 7975 1750 60  0000 C CNN
+	1    7975 1750
+	0    1    1    0
+$EndComp
+Wire Wire Line
+	8100 2075 8350 2075
+Wire Wire Line
+	8350 1750 8350 2425
+Wire Wire Line
+	8125 1750 8350 1750
+Connection ~ 8350 2075
+Wire Wire Line
+	7800 2075 7425 2075
+Wire Wire Line
+	7125 2075 5750 2075
+Wire Wire Line
+	7600 1475 7600 2075
+Wire Wire Line
+	7600 1750 7825 1750
+Connection ~ 7600 2075
+Wire Wire Line
+	7600 1475 8175 1475
+Connection ~ 7600 1750
 $EndSCHEMATC

Commit message: pre-net import
Parts:
- removed JP1, JP2: JUMPER, aero:Pin_Header_1x02_2mm, symbol JUMPER
- J2: footprint aero:Conn_Molex_78171-02 -> Pin_Headers:Pin_Header_Straight_1x02
Connections:
- net Vbatt: now also J2.1 (BATT+)
- net at C24.1, CON1.1 (VBUS): now also C23.1, U7.1 (IN)
Changed lines of the file:
@@
 F 0 "J2" H 5000 5900 60  0000 C CNN
 F 1 "LiPoly_Conn" H 5200 5400 60  0000 C CNN
-F 2 "aero:Conn_Molex_78171-02" H 5050 5500 60  0001 C CNN
+F 2 "Pin_Headers:Pin_Header_Straight_1x02" H 5050 5500 60  0001 C CNN
 F 3 "" H 5050 5500 60  0000 C CNN
 	1    5050 5500
@@
 	1    0    0    -1
 $EndComp
-$Comp
-L JUMPER JP1
-U 1 1 5540E544
-P 2700 3450
-F 0 "JP1" H 2700 3600 50  0000 C CNN
-F 1 "JUMPER" H 2700 3370 50  0000 C CNN
-F 2 "aero:Pin_Header_1x02_2mm" H 2700 3450 60  0001 C CNN
-F 3 "" H 2700 3450 60  0000 C CNN
-	1    2700 3450
-	0    1    1    0
-$EndComp
-$Comp
-L JUMPER JP2
-U 1 1 5540E5FA
-P 5250 4800
-F 0 "JP2" H 5250 4950 50  0000 C CNN
-F 1 "JUMPER" H 5250 4720 50  0000 C CNN
-F 2 "aero:Pin_Header_1x02_2mm" H 5250 4800 60  0001 C CNN
-F 3 "" H 5250 4800 60  0000 C CNN
-	1    5250 4800
-	0    1    1    0
-$EndComp
 Wire Wire Line
-	2700 3750 2700 4000
+	2700 2650 2700 4000
 Wire Wire Line
-	2700 3150 2700 2650
-Wire Wire Line
-	5250 5100 5250 5300
+	5250 4000 5250 5300
 Wire Wire Line
 	2350 2450 2350 2650
@@
 Connection ~ 5250 4000
 Wire Wire Line
-	5250 4000 5250 4500
-Wire Wire Line
 	4800 5150 4800 5050
